File: linectrlsingle.kicad_sch (KiCad schematic)
At the start: 32 parts, among them J1 6P4C, J3 6P4C, K1 Relay_SPST-NO, K3 Relay_SPDT, Q1 PMOS, Q3 PMOS, T1 Transformer_1P_1S

Commit message: place footprints for one line module
Parts:
- renumbered C3 to C2, C5 to C3, D3 to D2, D5 to D3, D7 to D4, J1 to J3, J3 to J4, K3 to K2, Q3 to Q2, R3 to R10, R4 to R11, R7 to R12, R9 to R13, R11 to R14, R13 to R15, R15 to R16, R1 to R9, TP1 to TP25, TP2 to TP26, TP5 to TP27, TP6 to TP28, TP9 to TP29, TP11 to TP30, TP13 to TP31, TP15 to TP32, TP17 to TP33

Commit message: layout and replicate remaining lines
Parts:
- R14, R15, R16: footprint Resistor_THT:R_Axial_DIN0207_L6.3mm_D2.5mm_P10.16mm_Horizontal -> Resistor_THT:R_Axial_DIN0207_L6.3mm_D2.5mm_P7.62mm_Horizontal
Changed lines of the file:
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@@
 			)
 		)
-		(property "Footprint" "Resistor_THT:R_Axial_DIN0207_L6.3mm_D2.5mm_P10.16mm_Horizontal"
+		(property "Footprint" "Resistor_THT:R_Axial_DIN0207_L6.3mm_D2.5mm_P7.62mm_Horizontal"
 			(at 201.168 109.22 90)
 			(hide yes)
@@
 			)
 		)
-		(property "Footprint" "Resistor_THT:R_Axial_DIN0207_L6.3mm_D2.5mm_P10.16mm_Horizontal"
+		(property "Footprint" "Resistor_THT:R_Axial_DIN0207_L6.3mm_D2.5mm_P7.62mm_Horizontal"
 			(at 165.862 80.01 90)
 			(hide yes)
@@
 			)
 		)
-		(property "Footprint" "Resistor_THT:R_Axial_DIN0207_L6.3mm_D2.5mm_P10.16mm_Horizontal"
+		(property "Footprint" "Resistor_THT:R_Axial_DIN0207_L6.3mm_D2.5mm_P7.62mm_Horizontal"
 			(at 174.752 78.74 90)
 			(hide yes)

Commit message: convert to 4 layer board and add power/gnd planes
Connections:
- net GND: no longer J4.SH
- net GNDD: now also J4.SH

Commit message: fix controlsw/hooksw subsheet error
Connections:
- net controlSW1 renamed controlSW
- net hookSW1 renamed hookSW
Changed lines of the file:
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@@
 		)
 	)
-	(hierarchical_label "hookSW1"
+	(hierarchical_label "hookSW"
 		(shape input)
 		(at 162.56 86.36 180)
@@
 		)
 	)
-	(hierarchical_label "controlSW1"
+	(hierarchical_label "controlSW"
 		(shape input)
 		(at 189.23 114.3 180)
