File: linectrlsingle.kicad_sch (KiCad schematic)
At the start: 36 parts, among them J5 6P4C, J6 6P4C, K1 Relay_SPST-NO, K2 Relay_SPDT, Q2 PMOS, Q3 PMOS, T1 Transformer_1P_1S

Commit message: nearly complete layout lol
Parts:
- D2, D3: value BAT54LT1G -> RB520S30T5G; footprint Package_TO_SOT_SMD:SOT-23 -> Diode_SMD:D_SOD-523; DKPN BAT54LT1GOSCT-ND -> RB520S30T5GOSCT-ND
Connections:
- net GND: now also T1.4 (SA); no longer T1.3 (SA)
- net at J5.3, J6.2, K1.6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: now also T1.3 (AB); no longer T1.2 (AB)
- net at C20.1, D2.2 (A), D3.1 (K)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: now also T1.6 (SB); no longer T1.4 (SB)
Changed lines of the file:
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@@
 			)
 		)
-		(property "Value" "BAT54LT1G"
+		(property "Value" "RB520S30T5G"
 			(at 91.44 92.7099 90)
 			(show_name no)
@@
 			)
 		)
-		(property "Footprint" "Package_TO_SOT_SMD:SOT-23"
+		(property "Footprint" "Diode_SMD:D_SOD-523"
 			(at 93.98 91.44 0)
 			(hide yes)
@@
 			)
 		)
-		(property "DKPN" "BAT54LT1GOSCT-ND"
+		(property "DKPN" "RB520S30T5GOSCT-ND"
 			(at 93.98 91.44 90)
 			(hide yes)
@@
 			)
 		)
-		(property "Value" "BAT54LT1G"
+		(property "Value" "RB520S30T5G"
 			(at 101.6 90.1701 90)
 			(show_name no)
@@
 			)
 		)
-		(property "Footprint" "Package_TO_SOT_SMD:SOT-23"
+		(property "Footprint" "Diode_SMD:D_SOD-523"
 			(at 99.06 91.44 0)
 			(hide yes)
@@
 			)
 		)
-		(property "DKPN" "BAT54LT1GOSCT-ND"
+		(property "DKPN" "RB520S30T5GOSCT-ND"
 			(at 99.06 91.44 90)
 			(hide yes)
@@
 		(pin "1"
 		)
-		(pin "2"
+		(pin "6"
 		)
 		(pin "4"
