File: pbx-sniffer-v2.kicad_pcb (KiCad board)
At the start: 2 copper layers, 390.2 x 170.1 mm, 297 parts, among them J1 6P4C, J10 6P4C, J11 6P4C, J12 6P4C, J13 6P4C, J14 6P4C, J15 6P4C, J16 6P4C, J17 8P8C, J18 8P8C, J2 6P4C, J3 6P4C, J4 6P4C, J5 6P4C, J6 6P4C, J7 6P4C, J8 6P4C, J9 6P4C, K1 Relay_SPST-NO, K10 Relay_SPST-NO, K11 Relay_SPDT, K12 Relay_SPDT, K13 Relay_SPST-NO, K14 Relay_SPST-NO, K15 Relay_SPDT, K16 Relay_SPDT, K2 Relay_SPST-NO, K3 Relay_SPDT, K4 Relay_SPDT, K5 Relay_SPST-NO, K6 Relay_SPST-NO, K7 Relay_SPDT, K8 Relay_SPDT, K9 Relay_SPST-NO, Q1 PMOS, Q10 PMOS, Q11 PMOS, Q12 PMOS, Q13 PMOS, Q14 PMOS, Q15 PMOS, Q16 PMOS, Q2 PMOS, Q3 PMOS, Q4 PMOS, Q5 PMOS, Q6 PMOS, Q7 PMOS, Q8 PMOS, Q9 PMOS, T1 Transformer_1P_1S, T2 Transformer_1P_1S, T3 Transformer_1P_1S, T4 Transformer_1P_1S, T5 Transformer_1P_1S, T6 Transformer_1P_1S, T7 Transformer_1P_1S, T8 Transformer_1P_1S, U1 STM32NucleoF303RE, U2 LM358, U3 LM358, U4 LM358, U5 LM358, U6 74LS165, U7 MCP3008

Commit message: make each phone line a subsheet and start redoing layout
Parts:
- removed C1, C10, C11, C12, C13, C14, C15, C16, C17, C18, C19, C2, C20, C21, C22, C23, C24, C3, C4, C5, C6, C7, C8, C9: 0.47u, Capacitor_THT:C_Rect_L7.0mm_W2.0mm_P5.00mm
- removed D1, D10, D11, D12, D13, D14, D15, D16, D17, D18, D19, D2, D20, D21, D22, D23, D24, D25, D26, D27, D28, D29, D3, D30, D31, D32, D4, D5, D6, D7, D8, D9: 1N4148, Diode_THT:D_DO-35_SOD27_P7.62mm_Horizontal
- removed J1, J10, J11, J12, J13, J14, J15, J16, J2, J3, J4, J5, J6, J7, J8, J9: 6P4C, Phones:CUI_CRJ050-1-TH
- removed JP1, JP2, JP3, JP4, JP5, JP6, JP7, JP8: Jumper_1-2, Jumper:SolderJumper-3_P1.3mm_Bridged2Bar12_RoundedPad1.0x1.5mm
- removed K1, K10, K13, K14, K2, K5, K6, K9: Relay_SPST-NO, Relay_THT:Relay_SPST_StandexMeder_SIL_Form1A
- removed K11, K12, K15, K16, K3, K4, K7, K8: Relay_SPDT, Phones:K_AZ943-1C_AMZ
- removed Q1, Q10, Q11, Q12, Q13, Q14, Q15, Q16, Q2, Q3, Q4, Q5, Q6, Q7, Q8, Q9: PMOS, Package_TO_SOT_THT:TO-92_HandSolder
- removed R1, R10, R17, R18, R19, R2, R20, R21, R22, R25, R26, R3, R33, R34, R35, R36, R37, R38, R4, R41, R42, R49, R5, R50, R51, R52, R53, R54, R57, R58, R6, R9: 10k, Resistor_THT:R_Axial_DIN0207_L6.3mm_D2.5mm_P7.62mm_Horizontal
- removed R11, R12, R15, R16, R27, R28, R31, R32, R43, R44, R47, R48, R59, R60, R63, R64: 10k, Resistor_THT:R_Axial_DIN0207_L6.3mm_D2.5mm_P10.16mm_Horizontal
- removed R13, R14, R29, R30, R45, R46, R61, R62: 500, Resistor_THT:R_Axial_DIN0207_L6.3mm_D2.5mm_P10.16mm_Horizontal
- removed R23, R24, R39, R40, R55, R56, R7, R8: 1k, Resistor_THT:R_Axial_DIN0207_L6.3mm_D2.5mm_P7.62mm_Horizontal
- removed T1, T2, T3, T4, T5, T6, T7, T8: Transformer_1P_1S, Phones:TY-145P
- removed TP1, TP10, TP11, TP12, TP13, TP14, TP15, TP16, TP17, TP18, TP19, TP2, TP20, TP21, TP22, TP23, TP24, TP25, TP26, TP27, TP28, TP29, TP3, TP30, TP31, TP32, TP33, TP34, TP35, TP36, TP37, TP38, TP39, TP4, TP40, TP41, TP42, TP43, TP44, TP45, TP46, TP47, TP48, TP49, TP5, TP50, TP51, TP52, TP53, TP54, TP55, TP56, TP57, TP58, TP59, TP6, TP60, TP61, TP62, TP63, TP64, TP65, TP66, TP67, TP68, TP69, TP7, TP70, TP71, TP72, TP8, TP9: TestPoint, Testpoints:M5_3in1_TestPoint
- removed U2, U3, U4, U5: LM358, Package_DIP:DIP-8_W7.62mm
Routing:
- net Net-(T8-AB): track 154.7 -> 0.00 mm, vias 2 -> 0
- net Net-(T6-AB): track 154.7 -> 0.00 mm, vias 2 -> 0
- net Net-(T4-AB): track 154.7 -> 0.00 mm, vias 2 -> 0
- net Net-(T2-AB): track 154.7 -> 0.00 mm, vias 2 -> 0
- net Net-(J5-Pad4): track 152.7 -> 0.00 mm
- net Net-(J1-Pad4): track 152.7 -> 0.00 mm
- net Net-(J11-Pad1): track 152.7 -> 0.00 mm
- net Net-(J13-Pad4): track 152.7 -> 0.00 mm
- net Net-(T7-AB): track 152.1 -> 0.00 mm, vias 2 -> 0
- net Net-(T5-AB): track 152.1 -> 0.00 mm, vias 2 -> 0
- net Net-(T1-AB): track 152.1 -> 0.00 mm, vias 2 -> 0
- net Net-(T3-AB): track 152.1 -> 0.00 mm, vias 2 -> 0
- net Net-(J2-Pad4): track 148.0 -> 0.00 mm
- net Net-(J14-Pad4): track 148.0 -> 0.00 mm
- net Net-(J10-Pad4): track 148.0 -> 0.00 mm
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
Commit message: place footprints for one line module
Parts:
- added C1: 0.47u, Capacitor_THT:C_Rect_L7.0mm_W2.0mm_P5.00mm, F.Cu at (189.4, 162.9)
- added C10: 0.47u, Capacitor_THT:C_Rect_L7.0mm_W2.0mm_P5.00mm, F.Cu at (-52.2, 71.1)
- added C11: 0.47u, Capacitor_THT:C_Rect_L7.0mm_W2.0mm_P5.00mm, F.Cu at (-52.2, 74.7)
- added C12: 0.47u, Capacitor_THT:C_Rect_L7.0mm_W2.0mm_P5.00mm, F.Cu at (-52.2, 78.2)
- added C13: 0.47u, Capacitor_THT:C_Rect_L7.0mm_W2.0mm_P5.00mm, F.Cu at (-184.7, 216.8)
- added C14: 0.47u, Capacitor_THT:C_Rect_L7.0mm_W2.0mm_P5.00mm, F.Cu at (-184.7, 220.3)
- added C15: 0.47u, Capacitor_THT:C_Rect_L7.0mm_W2.0mm_P5.00mm, F.Cu at (-184.7, 223.9)
- added C16: 0.47u, Capacitor_THT:C_Rect_L7.0mm_W2.0mm_P5.00mm, F.Cu at (-52.2, 188.6)
- added C17: 0.47u, Capacitor_THT:C_Rect_L7.0mm_W2.0mm_P5.00mm, F.Cu at (-52.2, 192.1)
- added C18: 0.47u, Capacitor_THT:C_Rect_L7.0mm_W2.0mm_P5.00mm, F.Cu at (-52.2, 195.7)
- added C19: 0.47u, Capacitor_THT:C_Rect_L7.0mm_W2.0mm_P5.00mm, F.Cu at (-114.6, 129.9)
- added C2: 0.47u, Capacitor_THT:C_Rect_L7.0mm_W2.0mm_P5.00mm, F.Cu at (192.8, 193.3)
- added C20: 0.47u, Capacitor_THT:C_Rect_L7.0mm_W2.0mm_P5.00mm, F.Cu at (-114.6, 133.4)
- added C21: 0.47u, Capacitor_THT:C_Rect_L7.0mm_W2.0mm_P5.00mm, F.Cu at (-114.6, 137.0)
- added C22: 0.47u, Capacitor_THT:C_Rect_L7.0mm_W2.0mm_P5.00mm, F.Cu at (-114.6, 71.1)
- added C23: 0.47u, Capacitor_THT:C_Rect_L7.0mm_W2.0mm_P5.00mm, F.Cu at (-114.6, 74.7)
- added C24: 0.47u, Capacitor_THT:C_Rect_L7.0mm_W2.0mm_P5.00mm, F.Cu at (-114.6, 78.2)
- added C3: 0.47u, Capacitor_THT:C_Rect_L7.0mm_W2.0mm_P5.00mm, F.Cu at (198.8, 219.9)
- added C4: 0.47u, Capacitor_THT:C_Rect_L7.0mm_W2.0mm_P5.00mm, F.Cu at (-52.2, 129.9)
- added C5: 0.47u, Capacitor_THT:C_Rect_L7.0mm_W2.0mm_P5.00mm, F.Cu at (-52.2, 133.4)
- added C6: 0.47u, Capacitor_THT:C_Rect_L7.0mm_W2.0mm_P5.00mm, F.Cu at (-52.2, 137.0)
- added C7: 0.47u, Capacitor_THT:C_Rect_L7.0mm_W2.0mm_P5.00mm, F.Cu at (-114.6, 247.3)
- added C8: 0.47u, Capacitor_THT:C_Rect_L7.0mm_W2.0mm_P5.00mm, F.Cu at (-114.6, 250.9)
- added C9: 0.47u, Capacitor_THT:C_Rect_L7.0mm_W2.0mm_P5.00mm, F.Cu at (-114.6, 254.4)
- added D1: 1N4148, Diode_THT:D_DO-35_SOD27_P7.62mm_Horizontal, F.Cu at (198.8, 200.7)
- added D10: 1N4148, Diode_THT:D_DO-35_SOD27_P7.62mm_Horizontal, F.Cu at (-114.8, 236.7)
- added D11: 1N4148, Diode_THT:D_DO-35_SOD27_P7.62mm_Horizontal, F.Cu at (-114.8, 240.2)
- added D12: 1N4148, Diode_THT:D_DO-35_SOD27_P7.62mm_Horizontal, F.Cu at (-114.8, 243.8)
- added D13: 1N4148, Diode_THT:D_DO-35_SOD27_P7.62mm_Horizontal, F.Cu at (-52.4, 56.9)
- added D14: 1N4148, Diode_THT:D_DO-35_SOD27_P7.62mm_Horizontal, F.Cu at (-52.4, 60.5)
- added D15: 1N4148, Diode_THT:D_DO-35_SOD27_P7.62mm_Horizontal, F.Cu at (-52.4, 64.0)
- added D16: 1N4148, Diode_THT:D_DO-35_SOD27_P7.62mm_Horizontal, F.Cu at (-52.4, 67.6)
- added D17: 1N4148, Diode_THT:D_DO-35_SOD27_P7.62mm_Horizontal, F.Cu at (-184.9, 202.6)
- added D18: 1N4148, Diode_THT:D_DO-35_SOD27_P7.62mm_Horizontal, F.Cu at (-184.9, 206.1)
- added D19: 1N4148, Diode_THT:D_DO-35_SOD27_P7.62mm_Horizontal, F.Cu at (-184.9, 209.7)
- added D2: 1N4148, Diode_THT:D_DO-35_SOD27_P7.62mm_Horizontal, F.Cu at (202.8, 193.1)
- added D20: 1N4148, Diode_THT:D_DO-35_SOD27_P7.62mm_Horizontal, F.Cu at (-184.9, 213.2)
- added D21: 1N4148, Diode_THT:D_DO-35_SOD27_P7.62mm_Horizontal, F.Cu at (-52.4, 174.4)
- added D22: 1N4148, Diode_THT:D_DO-35_SOD27_P7.62mm_Horizontal, F.Cu at (-52.4, 177.9)
- added D23: 1N4148, Diode_THT:D_DO-35_SOD27_P7.62mm_Horizontal, F.Cu at (-52.4, 181.5)
- added D24: 1N4148, Diode_THT:D_DO-35_SOD27_P7.62mm_Horizontal, F.Cu at (-52.4, 185.0)
- added D25: 1N4148, Diode_THT:D_DO-35_SOD27_P7.62mm_Horizontal, F.Cu at (-114.8, 115.7)
- added D26: 1N4148, Diode_THT:D_DO-35_SOD27_P7.62mm_Horizontal, F.Cu at (-114.8, 119.2)
- added D27: 1N4148, Diode_THT:D_DO-35_SOD27_P7.62mm_Horizontal, F.Cu at (-114.8, 122.8)
- added D28: 1N4148, Diode_THT:D_DO-35_SOD27_P7.62mm_Horizontal, F.Cu at (-114.8, 126.3)
- added D29: 1N4148, Diode_THT:D_DO-35_SOD27_P7.62mm_Horizontal, F.Cu at (-114.8, 56.9)
- added D3: 1N4148, Diode_THT:D_DO-35_SOD27_P7.62mm_Horizontal, F.Cu at (194.6, 224.8)
- added D30: 1N4148, Diode_THT:D_DO-35_SOD27_P7.62mm_Horizontal, F.Cu at (-114.8, 60.5)
- added D31: 1N4148, Diode_THT:D_DO-35_SOD27_P7.62mm_Horizontal, F.Cu at (-114.8, 64.0)
- added D32: 1N4148, Diode_THT:D_DO-35_SOD27_P7.62mm_Horizontal, F.Cu at (-114.8, 67.6)
- added D4: 1N4148, Diode_THT:D_DO-35_SOD27_P7.62mm_Horizontal, F.Cu at (194.6, 242.6)
- added D5: 1N4148, Diode_THT:D_DO-35_SOD27_P7.62mm_Horizontal, F.Cu at (-52.4, 115.7)
- added D6: 1N4148, Diode_THT:D_DO-35_SOD27_P7.62mm_Horizontal, F.Cu at (-52.4, 119.2)
- added D7: 1N4148, Diode_THT:D_DO-35_SOD27_P7.62mm_Horizontal, F.Cu at (-52.4, 122.8)
- added D8: 1N4148, Diode_THT:D_DO-35_SOD27_P7.62mm_Horizontal, F.Cu at (-52.4, 126.3)
- added D9: 1N4148, Diode_THT:D_DO-35_SOD27_P7.62mm_Horizontal, F.Cu at (-114.8, 233.1)
- added J1: 8P8C, Phones:AMPHENOL_54602-908LF, F.Cu at (-226.3, 126.2)
- added J10: 6P4C, Phones:CUI_CRJ050-1-TH, F.Cu at (-77.3, 34.6)
- added J11: 6P4C, Phones:CUI_CRJ050-1-TH, F.Cu at (-227.3, 180.2)
- added J12: 6P4C, Phones:CUI_CRJ050-1-TH, F.Cu at (-209.8, 180.2)
- added J13: 6P4C, Phones:CUI_CRJ050-1-TH, F.Cu at (-94.8, 152.0)
- added J14: 6P4C, Phones:CUI_CRJ050-1-TH, F.Cu at (-77.3, 152.0)
- added J15: 6P4C, Phones:CUI_CRJ050-1-TH, F.Cu at (-157.2, 93.3)
- added J16: 6P4C, Phones:CUI_CRJ050-1-TH, F.Cu at (-139.7, 93.3)
- added J2: 8P8C, Phones:AMPHENOL_54602-908LF, F.Cu at (-208.1, 126.2)
- added J3: 6P4C, Phones:CUI_CRJ050-1-TH, F.Cu at (195.0, 123.9)
- added J4: 6P4C, Phones:CUI_CRJ050-1-TH, F.Cu at (195.0, 276.9)
- added J5: 6P4C, Phones:CUI_CRJ050-1-TH, F.Cu at (-94.8, 93.3)
- added J6: 6P4C, Phones:CUI_CRJ050-1-TH, F.Cu at (-77.3, 93.3)
- added J7: 6P4C, Phones:CUI_CRJ050-1-TH, F.Cu at (-157.2, 210.8)
- added J8: 6P4C, Phones:CUI_CRJ050-1-TH, F.Cu at (-139.7, 210.8)
- added J9: 6P4C, Phones:CUI_CRJ050-1-TH, F.Cu at (-94.8, 34.6)
- added JP1: Jumper_1-2, Jumper:SolderJumper-3_P1.3mm_Bridged2Bar12_RoundedPad1.0x1.5mm, F.Cu at (189.3, 242.6)
- added JP2: Jumper_1-2, Jumper:SolderJumper-3_P1.3mm_Bridged2Bar12_RoundedPad1.0x1.5mm, F.Cu at (-80.1, 136.3)
- added JP3: Jumper_1-2, Jumper:SolderJumper-3_P1.3mm_Bridged2Bar12_RoundedPad1.0x1.5mm, F.Cu at (-142.5, 253.8)
- added JP4: Jumper_1-2, Jumper:SolderJumper-3_P1.3mm_Bridged2Bar12_RoundedPad1.0x1.5mm, F.Cu at (-80.1, 77.6)
- added JP5: Jumper_1-2, Jumper:SolderJumper-3_P1.3mm_Bridged2Bar12_RoundedPad1.0x1.5mm, F.Cu at (-212.7, 223.2)
- added JP6: Jumper_1-2, Jumper:SolderJumper-3_P1.3mm_Bridged2Bar12_RoundedPad1.0x1.5mm, F.Cu at (-80.1, 195.0)
- added JP7: Jumper_1-2, Jumper:SolderJumper-3_P1.3mm_Bridged2Bar12_RoundedPad1.0x1.5mm, F.Cu at (-142.5, 136.3)
- added JP8: Jumper_1-2, Jumper:SolderJumper-3_P1.3mm_Bridged2Bar12_RoundedPad1.0x1.5mm, F.Cu at (-142.5, 77.6)
- added K1: Relay_SPST-NO, Relay_THT:Relay_SPST_StandexMeder_SIL_Form1A, F.Cu at (199.8, 241.5)
- added K10: Relay_SPDT, Phones:K_AZ943-1C_AMZ, F.Cu at (-205.7, 203.1)
- added K11: Relay_SPST-NO, Relay_THT:Relay_SPST_StandexMeder_SIL_Form1A, F.Cu at (-65.4, 144.1)
- added K12: Relay_SPDT, Phones:K_AZ943-1C_AMZ, F.Cu at (-73.2, 174.8)
- added K13: Relay_SPST-NO, Relay_THT:Relay_SPST_StandexMeder_SIL_Form1A, F.Cu at (-127.8, 85.3)
- added K14: Relay_SPDT, Phones:K_AZ943-1C_AMZ, F.Cu at (-135.6, 116.1)
- added K15: Relay_SPST-NO, Relay_THT:Relay_SPST_StandexMeder_SIL_Form1A, F.Cu at (-127.8, 26.6)
- added K16: Relay_SPDT, Phones:K_AZ943-1C_AMZ, F.Cu at (-135.6, 57.4)
- added K2: Relay_SPDT, Phones:K_AZ943-1C_AMZ, F.Cu at (194.8, 246.2)
- added K3: Relay_SPST-NO, Relay_THT:Relay_SPST_StandexMeder_SIL_Form1A, F.Cu at (-65.4, 85.3)
- added K4: Relay_SPDT, Phones:K_AZ943-1C_AMZ, F.Cu at (-73.2, 116.1)
- added K5: Relay_SPST-NO, Relay_THT:Relay_SPST_StandexMeder_SIL_Form1A, F.Cu at (-127.8, 202.8)
- added K6: Relay_SPDT, Phones:K_AZ943-1C_AMZ, F.Cu at (-135.6, 233.6)
- added K7: Relay_SPST-NO, Relay_THT:Relay_SPST_StandexMeder_SIL_Form1A, F.Cu at (-65.4, 26.6)
- added K8: Relay_SPDT, Phones:K_AZ943-1C_AMZ, F.Cu at (-73.2, 57.4)
- added K9: Relay_SPST-NO, Relay_THT:Relay_SPST_StandexMeder_SIL_Form1A, F.Cu at (-197.9, 172.3)
- added Q1: PMOS, Package_TO_SOT_THT:TO-92_HandSolder, F.Cu at (186.5, 217.3)
- added Q10: PMOS, Package_TO_SOT_THT:TO-92_HandSolder, F.Cu at (-185.8, 185.3)
- added Q11: PMOS, Package_TO_SOT_THT:TO-92_HandSolder, F.Cu at (-53.2, 151.0)
- added Q12: PMOS, Package_TO_SOT_THT:TO-92_HandSolder, F.Cu at (-53.2, 157.1)
- added Q13: PMOS, Package_TO_SOT_THT:TO-92_HandSolder, F.Cu at (-115.6, 92.3)
- added Q14: PMOS, Package_TO_SOT_THT:TO-92_HandSolder, F.Cu at (-115.6, 98.4)
- added Q15: PMOS, Package_TO_SOT_THT:TO-92_HandSolder, F.Cu at (-115.6, 33.6)
- added Q16: PMOS, Package_TO_SOT_THT:TO-92_HandSolder, F.Cu at (-115.6, 39.7)
- added Q2: PMOS, Package_TO_SOT_THT:TO-92_HandSolder, F.Cu at (186.5, 223.4)
- added Q3: PMOS, Package_TO_SOT_THT:TO-92_HandSolder, F.Cu at (-53.2, 92.3)
- added Q4: PMOS, Package_TO_SOT_THT:TO-92_HandSolder, F.Cu at (-53.2, 98.4)
- added Q5: PMOS, Package_TO_SOT_THT:TO-92_HandSolder, F.Cu at (-115.6, 209.7)
- added Q6: PMOS, Package_TO_SOT_THT:TO-92_HandSolder, F.Cu at (-115.6, 215.8)
- added Q7: PMOS, Package_TO_SOT_THT:TO-92_HandSolder, F.Cu at (-53.2, 33.6)
- added Q8: PMOS, Package_TO_SOT_THT:TO-92_HandSolder, F.Cu at (-53.2, 39.7)
- added Q9: PMOS, Package_TO_SOT_THT:TO-92_HandSolder, F.Cu at (-185.8, 179.2)
- added R1: 10k, Resistor_THT:R_Axial_DIN0207_L6.3mm_D2.5mm_P10.16mm_Horizontal, F.Cu at (-234.5, 136.6)
- added R10: 10k, Resistor_THT:R_Axial_DIN0207_L6.3mm_D2.5mm_P7.62mm_Horizontal, F.Cu at (151.3, 215.0)
- added R11: 10k, Resistor_THT:R_Axial_DIN0207_L6.3mm_D2.5mm_P7.62mm_Horizontal, F.Cu at (187.4, 200.7)
- added R12: 1k, Resistor_THT:R_Axial_DIN0207_L6.3mm_D2.5mm_P7.62mm_Horizontal, F.Cu at (198.8, 211.2)
- added R13: 10k, Resistor_THT:R_Axial_DIN0207_L6.3mm_D2.5mm_P7.62mm_Horizontal, F.Cu at (192.8, 222.4)
- added R14: 10k, Resistor_THT:R_Axial_DIN0207_L6.3mm_D2.5mm_P10.16mm_Horizontal, F.Cu at (151.3, 219.2)
- added R15: 500, Resistor_THT:R_Axial_DIN0207_L6.3mm_D2.5mm_P10.16mm_Horizontal, F.Cu at (194.0, 151.9)
- added R16: 10k, Resistor_THT:R_Axial_DIN0207_L6.3mm_D2.5mm_P10.16mm_Horizontal, F.Cu at (151.3, 243.8)
- added R17: 10k, Resistor_THT:R_Axial_DIN0207_L6.3mm_D2.5mm_P7.62mm_Horizontal, F.Cu at (-63.2, 115.9)
- added R18: 10k, Resistor_THT:R_Axial_DIN0207_L6.3mm_D2.5mm_P7.62mm_Horizontal, F.Cu at (-63.2, 120.0)
- added R19: 10k, Resistor_THT:R_Axial_DIN0207_L6.3mm_D2.5mm_P7.62mm_Horizontal, F.Cu at (-63.2, 124.0)
- added R2: 10k, Resistor_THT:R_Axial_DIN0207_L6.3mm_D2.5mm_P10.16mm_Horizontal, F.Cu at (-234.5, 140.6)
- added R20: 1k, Resistor_THT:R_Axial_DIN0207_L6.3mm_D2.5mm_P7.62mm_Horizontal, F.Cu at (-63.2, 128.1)
- added R21: 10k, Resistor_THT:R_Axial_DIN0207_L6.3mm_D2.5mm_P7.62mm_Horizontal, F.Cu at (-63.2, 132.1)
- added R22: 10k, Resistor_THT:R_Axial_DIN0207_L6.3mm_D2.5mm_P10.16mm_Horizontal, F.Cu at (-67.0, 90.7)
- added R23: 500, Resistor_THT:R_Axial_DIN0207_L6.3mm_D2.5mm_P10.16mm_Horizontal, F.Cu at (-67.0, 94.8)
- added R24: 10k, Resistor_THT:R_Axial_DIN0207_L6.3mm_D2.5mm_P10.16mm_Horizontal, F.Cu at (-67.0, 98.8)
- added R25: 10k, Resistor_THT:R_Axial_DIN0207_L6.3mm_D2.5mm_P7.62mm_Horizontal, F.Cu at (-125.5, 233.4)
- added R26: 10k, Resistor_THT:R_Axial_DIN0207_L6.3mm_D2.5mm_P7.62mm_Horizontal, F.Cu at (-125.5, 237.4)
- added R27: 10k, Resistor_THT:R_Axial_DIN0207_L6.3mm_D2.5mm_P7.62mm_Horizontal, F.Cu at (-125.5, 241.5)
- added R28: 1k, Resistor_THT:R_Axial_DIN0207_L6.3mm_D2.5mm_P7.62mm_Horizontal, F.Cu at (-125.5, 245.5)
- added R29: 10k, Resistor_THT:R_Axial_DIN0207_L6.3mm_D2.5mm_P7.62mm_Horizontal, F.Cu at (-125.5, 249.6)
- added R3: 10k, Resistor_THT:R_Axial_DIN0207_L6.3mm_D2.5mm_P10.16mm_Horizontal, F.Cu at (-234.5, 144.7)
- added R30: 10k, Resistor_THT:R_Axial_DIN0207_L6.3mm_D2.5mm_P10.16mm_Horizontal, F.Cu at (-129.3, 208.2)
- added R31: 500, Resistor_THT:R_Axial_DIN0207_L6.3mm_D2.5mm_P10.16mm_Horizontal, F.Cu at (-129.3, 212.2)
- added R32: 10k, Resistor_THT:R_Axial_DIN0207_L6.3mm_D2.5mm_P10.16mm_Horizontal, F.Cu at (-129.3, 216.3)
- added R33: 10k, Resistor_THT:R_Axial_DIN0207_L6.3mm_D2.5mm_P7.62mm_Horizontal, F.Cu at (-63.2, 57.2)
- added R34: 10k, Resistor_THT:R_Axial_DIN0207_L6.3mm_D2.5mm_P7.62mm_Horizontal, F.Cu at (-63.2, 61.2)
- added R35: 10k, Resistor_THT:R_Axial_DIN0207_L6.3mm_D2.5mm_P7.62mm_Horizontal, F.Cu at (-63.2, 65.3)
- added R36: 1k, Resistor_THT:R_Axial_DIN0207_L6.3mm_D2.5mm_P7.62mm_Horizontal, F.Cu at (-63.2, 69.3)
- added R37: 10k, Resistor_THT:R_Axial_DIN0207_L6.3mm_D2.5mm_P7.62mm_Horizontal, F.Cu at (-63.2, 73.4)
- added R38: 10k, Resistor_THT:R_Axial_DIN0207_L6.3mm_D2.5mm_P10.16mm_Horizontal, F.Cu at (-67.0, 32.0)
- added R39: 500, Resistor_THT:R_Axial_DIN0207_L6.3mm_D2.5mm_P10.16mm_Horizontal, F.Cu at (-67.0, 36.1)
- added R4: 10k, Resistor_THT:R_Axial_DIN0207_L6.3mm_D2.5mm_P10.16mm_Horizontal, F.Cu at (-234.5, 148.7)
- added R40: 10k, Resistor_THT:R_Axial_DIN0207_L6.3mm_D2.5mm_P10.16mm_Horizontal, F.Cu at (-67.0, 40.1)
- added R41: 10k, Resistor_THT:R_Axial_DIN0207_L6.3mm_D2.5mm_P7.62mm_Horizontal, F.Cu at (-195.7, 202.8)
- added R42: 10k, Resistor_THT:R_Axial_DIN0207_L6.3mm_D2.5mm_P7.62mm_Horizontal, F.Cu at (-195.7, 206.9)
- added R43: 10k, Resistor_THT:R_Axial_DIN0207_L6.3mm_D2.5mm_P7.62mm_Horizontal, F.Cu at (-195.7, 210.9)
- added R44: 1k, Resistor_THT:R_Axial_DIN0207_L6.3mm_D2.5mm_P7.62mm_Horizontal, F.Cu at (-195.7, 215.0)
- added R45: 10k, Resistor_THT:R_Axial_DIN0207_L6.3mm_D2.5mm_P7.62mm_Horizontal, F.Cu at (-195.7, 219.0)
- added R46: 10k, Resistor_THT:R_Axial_DIN0207_L6.3mm_D2.5mm_P10.16mm_Horizontal, F.Cu at (-199.5, 177.7)
- added R47: 500, Resistor_THT:R_Axial_DIN0207_L6.3mm_D2.5mm_P10.16mm_Horizontal, F.Cu at (-199.5, 181.7)
- added R48: 10k, Resistor_THT:R_Axial_DIN0207_L6.3mm_D2.5mm_P10.16mm_Horizontal, F.Cu at (-199.5, 185.8)
- added R49: 10k, Resistor_THT:R_Axial_DIN0207_L6.3mm_D2.5mm_P7.62mm_Horizontal, F.Cu at (-63.2, 174.6)
- added R5: 10k, Resistor_THT:R_Axial_DIN0207_L6.3mm_D2.5mm_P10.16mm_Horizontal, F.Cu at (-234.5, 152.8)
- added R50: 10k, Resistor_THT:R_Axial_DIN0207_L6.3mm_D2.5mm_P7.62mm_Horizontal, F.Cu at (-63.2, 178.7)
- added R51: 10k, Resistor_THT:R_Axial_DIN0207_L6.3mm_D2.5mm_P7.62mm_Horizontal, F.Cu at (-63.2, 182.7)
- added R52: 1k, Resistor_THT:R_Axial_DIN0207_L6.3mm_D2.5mm_P7.62mm_Horizontal, F.Cu at (-63.2, 186.8)
- added R53: 10k, Resistor_THT:R_Axial_DIN0207_L6.3mm_D2.5mm_P7.62mm_Horizontal, F.Cu at (-63.2, 190.8)
- added R54: 10k, Resistor_THT:R_Axial_DIN0207_L6.3mm_D2.5mm_P10.16mm_Horizontal, F.Cu at (-67.0, 149.4)
- added R55: 500, Resistor_THT:R_Axial_DIN0207_L6.3mm_D2.5mm_P10.16mm_Horizontal, F.Cu at (-67.0, 153.5)
- added R56: 10k, Resistor_THT:R_Axial_DIN0207_L6.3mm_D2.5mm_P10.16mm_Horizontal, F.Cu at (-67.0, 157.5)
- added R57: 10k, Resistor_THT:R_Axial_DIN0207_L6.3mm_D2.5mm_P7.62mm_Horizontal, F.Cu at (-125.5, 115.9)
- added R58: 10k, Resistor_THT:R_Axial_DIN0207_L6.3mm_D2.5mm_P7.62mm_Horizontal, F.Cu at (-125.5, 120.0)
- added R59: 10k, Resistor_THT:R_Axial_DIN0207_L6.3mm_D2.5mm_P7.62mm_Horizontal, F.Cu at (-125.5, 124.0)
- added R6: 10k, Resistor_THT:R_Axial_DIN0207_L6.3mm_D2.5mm_P10.16mm_Horizontal, F.Cu at (-234.5, 156.8)
- added R60: 1k, Resistor_THT:R_Axial_DIN0207_L6.3mm_D2.5mm_P7.62mm_Horizontal, F.Cu at (-125.5, 128.1)
- added R61: 10k, Resistor_THT:R_Axial_DIN0207_L6.3mm_D2.5mm_P7.62mm_Horizontal, F.Cu at (-125.5, 132.1)
- added R62: 10k, Resistor_THT:R_Axial_DIN0207_L6.3mm_D2.5mm_P10.16mm_Horizontal, F.Cu at (-129.3, 90.7)
- added R63: 500, Resistor_THT:R_Axial_DIN0207_L6.3mm_D2.5mm_P10.16mm_Horizontal, F.Cu at (-129.3, 94.8)
- added R64: 10k, Resistor_THT:R_Axial_DIN0207_L6.3mm_D2.5mm_P10.16mm_Horizontal, F.Cu at (-129.3, 98.8)
- added R7: 10k, Resistor_THT:R_Axial_DIN0207_L6.3mm_D2.5mm_P10.16mm_Horizontal, F.Cu at (-234.5, 160.9)
- added R8: 10k, Resistor_THT:R_Axial_DIN0207_L6.3mm_D2.5mm_P10.16mm_Horizontal, F.Cu at (-234.5, 164.9)
- added R9: 10k, Resistor_THT:R_Axial_DIN0207_L6.3mm_D2.5mm_P7.62mm_Horizontal, F.Cu at (189.4, 151.9)
- added T1: Transformer_1P_1S, Phones:TY-145P, F.Cu at (194.7, 180.0)
- added T2: Transformer_1P_1S, Phones:TY-145P, F.Cu at (-92.6, 125.0)
- added T3: Transformer_1P_1S, Phones:TY-145P, F.Cu at (-155.0, 242.4)
- added T4: Transformer_1P_1S, Phones:TY-145P, F.Cu at (-92.6, 66.3)
- added T5: Transformer_1P_1S, Phones:TY-145P, F.Cu at (-225.1, 211.9)
- added T6: Transformer_1P_1S, Phones:TY-145P, F.Cu at (-92.6, 183.7)
- added T7: Transformer_1P_1S, Phones:TY-145P, F.Cu at (-155.0, 125.0)
- added T8: Transformer_1P_1S, Phones:TY-145P, F.Cu at (-155.0, 66.3)
- added TP1: TestPoint, Testpoints:M5_3in1_TestPoint, F.Cu at (-234.8, 104.6)
- added TP10: TestPoint, Testpoints:M5_3in1_TestPoint, F.Cu at (-193.0, 104.6)
- added TP11: TestPoint, Testpoints:M5_3in1_TestPoint, F.Cu at (-188.3, 104.6)
- added TP12: TestPoint, Testpoints:M5_3in1_TestPoint, F.Cu at (-183.7, 104.6)
- added TP13: TestPoint, Testpoints:M5_3in1_TestPoint, F.Cu at (-102.3, 200.4)
- added TP14: TestPoint, Testpoints:M5_3in1_TestPoint, F.Cu at (-97.6, 200.4)
- added TP15: TestPoint, Testpoints:M5_3in1_TestPoint, F.Cu at (-93.0, 200.4)
- added TP16: TestPoint, Testpoints:M5_3in1_TestPoint, F.Cu at (-88.3, 200.4)
- added TP17: TestPoint, Testpoints:M5_3in1_TestPoint, F.Cu at (-83.7, 200.4)
- added TP18: TestPoint, Testpoints:M5_3in1_TestPoint, F.Cu at (-79.0, 200.4)
- added TP19: TestPoint, Testpoints:M5_3in1_TestPoint, F.Cu at (-74.4, 200.4)
- added TP2: TestPoint, Testpoints:M5_3in1_TestPoint, F.Cu at (-230.2, 104.6)
- added TP20: TestPoint, Testpoints:M5_3in1_TestPoint, F.Cu at (-69.7, 200.4)
- added TP21: TestPoint, Testpoints:M5_3in1_TestPoint, F.Cu at (-65.1, 200.4)
- added TP22: TestPoint, Testpoints:M5_3in1_TestPoint, F.Cu at (-60.4, 200.4)
- added TP23: TestPoint, Testpoints:M5_3in1_TestPoint, F.Cu at (-55.8, 200.4)
- added TP24: TestPoint, Testpoints:M5_3in1_TestPoint, F.Cu at (-51.1, 200.4)
- added TP25: TestPoint, Testpoints:M5_3in1_TestPoint, F.Cu at (187.4, 136.0)
- added TP26: TestPoint, Testpoints:M5_3in1_TestPoint, F.Cu at (200.6, 136.0)
- added TP27: TestPoint, Testpoints:M5_3in1_TestPoint, F.Cu at (191.8, 136.0)
- added TP28: TestPoint, Testpoints:M5_3in1_TestPoint, F.Cu at (196.2, 136.0)
- added TP29: TestPoint, Testpoints:M5_3in1_TestPoint, F.Cu at (199.2, 158.8)
- added TP3: TestPoint, Testpoints:M5_3in1_TestPoint, F.Cu at (-225.5, 104.6)
- added TP30: TestPoint, Testpoints:M5_3in1_TestPoint, F.Cu at (191.7, 203.0)
- added TP31: TestPoint, Testpoints:M5_3in1_TestPoint, F.Cu at (186.1, 203.5)
- added TP32: TestPoint, Testpoints:M5_3in1_TestPoint, F.Cu at (186.8, 226.4)
- added TP33: TestPoint, Testpoints:M5_3in1_TestPoint, F.Cu at (190.4, 226.4)
- added TP34: TestPoint, Testpoints:M5_3in1_TestPoint, F.Cu at (-102.3, 103.2)
- added TP35: TestPoint, Testpoints:M5_3in1_TestPoint, F.Cu at (-97.6, 103.2)
- added TP36: TestPoint, Testpoints:M5_3in1_TestPoint, F.Cu at (-93.0, 103.2)
- added TP37: TestPoint, Testpoints:M5_3in1_TestPoint, F.Cu at (-88.3, 103.2)
- added TP38: TestPoint, Testpoints:M5_3in1_TestPoint, F.Cu at (-83.7, 103.2)
- added TP39: TestPoint, Testpoints:M5_3in1_TestPoint, F.Cu at (-79.0, 103.2)
- added TP4: TestPoint, Testpoints:M5_3in1_TestPoint, F.Cu at (-220.9, 104.6)
- added TP40: TestPoint, Testpoints:M5_3in1_TestPoint, F.Cu at (-74.4, 103.2)
- added TP41: TestPoint, Testpoints:M5_3in1_TestPoint, F.Cu at (-69.7, 103.2)
- added TP42: TestPoint, Testpoints:M5_3in1_TestPoint, F.Cu at (-65.1, 103.2)
- added TP43: TestPoint, Testpoints:M5_3in1_TestPoint, F.Cu at (-164.7, 220.6)
- added TP44: TestPoint, Testpoints:M5_3in1_TestPoint, F.Cu at (-160.0, 220.6)
- added TP45: TestPoint, Testpoints:M5_3in1_TestPoint, F.Cu at (-155.4, 220.6)
- added TP46: TestPoint, Testpoints:M5_3in1_TestPoint, F.Cu at (-150.7, 220.6)
- added TP47: TestPoint, Testpoints:M5_3in1_TestPoint, F.Cu at (-146.1, 220.6)
- added TP48: TestPoint, Testpoints:M5_3in1_TestPoint, F.Cu at (-141.4, 220.6)
- added TP49: TestPoint, Testpoints:M5_3in1_TestPoint, F.Cu at (-136.8, 220.6)
- added TP5: TestPoint, Testpoints:M5_3in1_TestPoint, F.Cu at (-216.2, 104.6)
- added TP50: TestPoint, Testpoints:M5_3in1_TestPoint, F.Cu at (-132.1, 220.6)
- added TP51: TestPoint, Testpoints:M5_3in1_TestPoint, F.Cu at (-127.5, 220.6)
- added TP52: TestPoint, Testpoints:M5_3in1_TestPoint, F.Cu at (-102.3, 44.5)
- added TP53: TestPoint, Testpoints:M5_3in1_TestPoint, F.Cu at (-97.6, 44.5)
- added TP54: TestPoint, Testpoints:M5_3in1_TestPoint, F.Cu at (-93.0, 44.5)
- added TP55: TestPoint, Testpoints:M5_3in1_TestPoint, F.Cu at (-88.3, 44.5)
- added TP56: TestPoint, Testpoints:M5_3in1_TestPoint, F.Cu at (-83.7, 44.5)
- added TP57: TestPoint, Testpoints:M5_3in1_TestPoint, F.Cu at (-79.0, 44.5)
- added TP58: TestPoint, Testpoints:M5_3in1_TestPoint, F.Cu at (-74.4, 44.5)
- added TP59: TestPoint, Testpoints:M5_3in1_TestPoint, F.Cu at (-69.7, 44.5)
- added TP6: TestPoint, Testpoints:M5_3in1_TestPoint, F.Cu at (-211.6, 104.6)
- added TP60: TestPoint, Testpoints:M5_3in1_TestPoint, F.Cu at (-65.1, 44.5)
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Connections:
- J17 pad 1: /TransferBtns/TBTN1 -> Net-(J17-Pad1)
- J17 pad 2: /TransferBtns/TBTN2 -> Net-(JP8-C)
- J17 pad 3: /TransferBtns/TBTN3 -> Net-(T8-AB)
- J17 pad 4: /TransferBtns/TBTN4 -> Net-(J17-Pad4)
- J18 pad 1: unconnected-(J18-Pad1) -> Net-(J17-Pad4)
- J18 pad 2: unconnected-(J18-Pad2) -> Net-(T8-AB)
- J18 pad 3: unconnected-(J18-Pad3) -> Net-(J18-Pad3)
- J18 pad 4: unconnected-(J18-Pad4) -> Net-(J17-Pad1)
- R65 pad 1: /TransferBtns/TBTN8 -> Net-(JP8-C)
- R65 pad 2: GNDD -> Net-(C22-Pad1)
- R66 pad 1: /TransferBtns/TBTN7 -> /LineCtrl4/LineCtrlSingle1/ampV+
- R66 pad 2: GNDD -> +5VA
- R67 pad 1: /TransferBtns/TBTN6 -> GND
- R67 pad 2: GNDD -> /LineCtrl4/LineCtrlSingle1/ampV+
- R68 pad 1: /TransferBtns/TBTN5 -> Net-(C24-Pad2)
- R68 pad 2: GNDD -> /LineCtrl4/LineCtrlSingle1/ampV-
- R69 pad 1: /TransferBtns/TBTN4 -> /LineCtrl4/LineCtrlSingle1/ampV-
- R69 pad 2: GNDD -> /ADC/adcCH7
- R70 pad 1: /TransferBtns/TBTN3 -> +5V
- R70 pad 2: GNDD -> /LineCtrl4/LineCtrlSingle1/hookSW1
- R71 pad 1: /TransferBtns/TBTN2 -> Net-(JP8-C)
- R71 pad 2: GNDD -> Net-(K15-Pad5)
- R72 pad 1: /TransferBtns/TBTN1 -> /LineCtrl4/LineCtrlSingle1/controlSW1
- R72 pad 2: GNDD -> +5V
- TP73 pad 1: /TransferBtns/TBTN8 -> Net-(T6-AB)
- TP74 pad 1: /TransferBtns/TBTN7 -> Net-(D21-A)
- TP75 pad 1: /TransferBtns/TBTN6 -> /LineCtrl2/LineCtrlSingle1/ampV+
- TP76 pad 1: /TransferBtns/TBTN5 -> /LineCtrl2/LineCtrlSingle1/hookSW1
- TP77 pad 1: /TransferBtns/TBTN4 -> /LineCtrl2/LineCtrlSingle1/controlSW1
- TP78 pad 1: /TransferBtns/TBTN3 -> Net-(J14-Pad3)
- TP79 pad 1: /TransferBtns/TBTN2 -> Net-(J15-Pad1)
- TP80 pad 1: /TransferBtns/TBTN1 -> Net-(J15-Pad4)
- TP81 pad 1: /TransferBtns/shiftClk -> Net-(JP7-C)
- TP82 pad 1: /TransferBtns/shiftInh -> Net-(T7-AB)
- TP83 pad 1: /TransferBtns/shiftLd -> Net-(D25-A)
- TP84 pad 1: /TransferBtns/shiftOut -> /LineCtrl3/LineCtrlSingle1/ampV+
- TP85 pad 1: /ADC/adcCH1 -> /LineCtrl3/LineCtrlSingle1/hookSW1
- TP86 pad 1: /ADC/adcCH2 -> /LineCtrl3/LineCtrlSingle1/controlSW1
- TP87 pad 1: /ADC/adcCH3 -> Net-(J16-Pad3)
- TP88 pad 1: /ADC/adcCH4 -> Net-(J17-Pad1)
- TP89 pad 1: /ADC/adcCH5 -> Net-(J17-Pad4)
- TP90 pad 1: /ADC/adcCH6 -> Net-(JP8-C)
- TP91 pad 1: /ADC/adcCH7 -> Net-(T8-AB)
- TP92 pad 1: /ADC/adcCH8 -> Net-(D29-A)
- TP93 pad 1: /SPI.spi0clk -> /LineCtrl4/LineCtrlSingle1/ampV+
- TP94 pad 1: /SPI.spi0miso -> /LineCtrl4/LineCtrlSingle1/hookSW1
- TP95 pad 1: /SPI.spi0mosi -> /LineCtrl4/LineCtrlSingle1/controlSW1
- TP96 pad 1: /SPI.spi0cs0 -> Net-(J18-Pad3)
Other:
- board text removed: "1"
- board text removed: "2"
- board text removed: "3"
- board text removed: "4"
- board text removed: "5"
- board text removed: "6"
- board text removed: "7"
- board text removed: "8"
- board text removed: "ADC Channels 1-8"
- board text removed: "SPI Lines"
- board text removed: "clk"
- board text removed: "cs"
- board text removed: "miso"
- board text removed: "mosi"

Commit message: layout and replicate remaining lines
Parts:
- added U2: LM358, Package_DIP:DIP-8_W7.62mm, F.Cu at (159.6, 192.4)
- added U3: LM358, Package_DIP:DIP-8_W7.62mm, F.Cu at (159.6, 178.8)
- added U4: LM358, Package_DIP:DIP-8_W7.62mm, F.Cu at (159.6, 165.2)
- added U5: LM358, Package_DIP:DIP-8_W7.62mm, F.Cu at (159.6, 151.6)
- R1, R14, R15, R16, R2, R22, R23, R24, R3, R4, R5, R6, R7, R8: footprint Resistor_THT:R_Axial_DIN0207_L6.3mm_D2.5mm_P10.16mm_Horizontal -> Resistor_THT:R_Axial_DIN0207_L6.3mm_D2.5mm_P7.62mm_Horizontal
- R30: renamed from R54; footprint Resistor_THT:R_Axial_DIN0207_L6.3mm_D2.5mm_P10.16mm_Horizontal -> Resistor_THT:R_Axial_DIN0207_L6.3mm_D2.5mm_P7.62mm_Horizontal
- R31: renamed from R55; footprint Resistor_THT:R_Axial_DIN0207_L6.3mm_D2.5mm_P10.16mm_Horizontal -> Resistor_THT:R_Axial_DIN0207_L6.3mm_D2.5mm_P7.62mm_Horizontal
- R32: renamed from R56; footprint Resistor_THT:R_Axial_DIN0207_L6.3mm_D2.5mm_P10.16mm_Horizontal -> Resistor_THT:R_Axial_DIN0207_L6.3mm_D2.5mm_P7.62mm_Horizontal
- R38: renamed from R30; footprint Resistor_THT:R_Axial_DIN0207_L6.3mm_D2.5mm_P10.16mm_Horizontal -> Resistor_THT:R_Axial_DIN0207_L6.3mm_D2.5mm_P7.62mm_Horizontal
- R39: renamed from R31; footprint Resistor_THT:R_Axial_DIN0207_L6.3mm_D2.5mm_P10.16mm_Horizontal -> Resistor_THT:R_Axial_DIN0207_L6.3mm_D2.5mm_P7.62mm_Horizontal
- R40: renamed from R32; footprint Resistor_THT:R_Axial_DIN0207_L6.3mm_D2.5mm_P10.16mm_Horizontal -> Resistor_THT:R_Axial_DIN0207_L6.3mm_D2.5mm_P7.62mm_Horizontal
- R46: renamed from R62; footprint Resistor_THT:R_Axial_DIN0207_L6.3mm_D2.5mm_P10.16mm_Horizontal -> Resistor_THT:R_Axial_DIN0207_L6.3mm_D2.5mm_P7.62mm_Horizontal
- R47: renamed from R63; footprint Resistor_THT:R_Axial_DIN0207_L6.3mm_D2.5mm_P10.16mm_Horizontal -> Resistor_THT:R_Axial_DIN0207_L6.3mm_D2.5mm_P7.62mm_Horizontal
- R48: renamed from R64; footprint Resistor_THT:R_Axial_DIN0207_L6.3mm_D2.5mm_P10.16mm_Horizontal -> Resistor_THT:R_Axial_DIN0207_L6.3mm_D2.5mm_P7.62mm_Horizontal
- R54: renamed from R38; footprint Resistor_THT:R_Axial_DIN0207_L6.3mm_D2.5mm_P10.16mm_Horizontal -> Resistor_THT:R_Axial_DIN0207_L6.3mm_D2.5mm_P7.62mm_Horizontal
- R55: renamed from R39; footprint Resistor_THT:R_Axial_DIN0207_L6.3mm_D2.5mm_P10.16mm_Horizontal -> Resistor_THT:R_Axial_DIN0207_L6.3mm_D2.5mm_P7.62mm_Horizontal
- R56: renamed from R40; footprint Resistor_THT:R_Axial_DIN0207_L6.3mm_D2.5mm_P10.16mm_Horizontal -> Resistor_THT:R_Axial_DIN0207_L6.3mm_D2.5mm_P7.62mm_Horizontal
- R62: renamed from R70; footprint Resistor_THT:R_Axial_DIN0207_L6.3mm_D2.5mm_P10.16mm_Horizontal -> Resistor_THT:R_Axial_DIN0207_L6.3mm_D2.5mm_P7.62mm_Horizontal
- R63: renamed from R71; footprint Resistor_THT:R_Axial_DIN0207_L6.3mm_D2.5mm_P10.16mm_Horizontal -> Resistor_THT:R_Axial_DIN0207_L6.3mm_D2.5mm_P7.62mm_Horizontal
- R64: renamed from R72; footprint Resistor_THT:R_Axial_DIN0207_L6.3mm_D2.5mm_P10.16mm_Horizontal -> Resistor_THT:R_Axial_DIN0207_L6.3mm_D2.5mm_P7.62mm_Horizontal
- R70: renamed from R46; footprint Resistor_THT:R_Axial_DIN0207_L6.3mm_D2.5mm_P10.16mm_Horizontal -> Resistor_THT:R_Axial_DIN0207_L6.3mm_D2.5mm_P7.62mm_Horizontal
- R71: renamed from R47; footprint Resistor_THT:R_Axial_DIN0207_L6.3mm_D2.5mm_P10.16mm_Horizontal -> Resistor_THT:R_Axial_DIN0207_L6.3mm_D2.5mm_P7.62mm_Horizontal
- R72: renamed from R48; footprint Resistor_THT:R_Axial_DIN0207_L6.3mm_D2.5mm_P10.16mm_Horizontal -> Resistor_THT:R_Axial_DIN0207_L6.3mm_D2.5mm_P7.62mm_Horizontal
- moved J1 599.5 mm to (373.0, 142.7), turned to 90 degrees
- moved TP1 598.6 mm to (357.1, 193.9), turned to -90 degrees
- moved TP2 594.8 mm to (357.1, 198.5), turned to -90 degrees
- moved TP3 590.9 mm to (357.1, 203.2), turned to -90 degrees
- moved TP4 587.1 mm to (357.1, 207.8), turned to -90 degrees
- moved R1 583.6 mm to (348.6, 160.8)
- moved R2 583.6 mm to (348.6, 164.9)
- moved R3 583.6 mm to (348.6, 168.9)
- moved R4 583.6 mm to (348.6, 173.0)
- moved R5 583.6 mm to (348.6, 177.1)
- moved R6 583.6 mm to (348.6, 181.1)
- moved R7 583.6 mm to (348.6, 185.2)
- moved R8 583.6 mm to (348.6, 189.2)
- moved TP5 583.4 mm to (357.1, 212.5), turned to -90 degrees
- moved J2 582.2 mm to (373.0, 161.5), turned to 90 degrees
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- renumbered C7 to C10, C8 to C11, C9 to C12, C19 to C13, C20 to C14, C21 to C15, C10 to C16, C11 to C17, C12 to C18, C22 to C19, C23 to C20, C24 to C21, C13 to C22, C14 to C23, C15 to C24, C16 to C7, C17 to C8, C18 to C9, D22 to D10, D23 to D11, D24 to D12, D9 to D13, D10 to D14, D11 to D15, D12 to D16, D25 to D17, D26 to D18, D27 to D19, D28 to D20, D13 to D21, D14 to D22, D15 to D23, D16 to D24, D29 to D25, D30 to D26, D31 to D27, D32 to D28, D17 to D29, D18 to D30, D19 to D31, D20 to D32, D21 to D9, J8 to J10, J15 to J11, J16 to J12, J9 to J13, J10 to J14, J17 to J15, J18 to J16, J11 to J17, J12 to J18, J13 to J7, J14 to J8, J7 to J9, JP6 to JP3, JP3 to JP4, JP7 to JP5, JP4 to JP6, JP8 to JP7, JP5 to JP8, K14 to K10, K7 to K11, K8 to K12, K15 to K13, K16 to K14, K9 to K15, K10 to K16, K11 to K5, K12 to K6, K5 to K7, K6 to K8, K13 to K9, Q14 to Q10, Q7 to Q11, Q8 to Q12, Q15 to Q13, Q16 to Q14, Q9 to Q15, Q10 to Q16, Q11 to Q5, Q12 to Q6, Q5 to Q7, Q6 to Q8, Q13 to Q9, R49 to R25, R50 to R26, R51 to R27, R52 to R28, R53 to R29, R25 to R33, R26 to R34, R27 to R35, R28 to R36, R29 to R37, R57 to R41, R58 to R42, R59 to R43, R60 to R44, R61 to R45, R33 to R49, R34 to R50, R35 to R51, R36 to R52, R37 to R53, R65 to R57, R66 to R58, R67 to R59, R68 to R60, R69 to R61, R41 to R65, R42 to R66, R43 to R67, R44 to R68, R45 to R69, T6 to T3, T3 to T4, T7 to T5, T4 to T6, T8 to T7, T5 to T8, TP70 to TP43, TP71 to TP44, TP72 to TP45, TP73 to TP46, TP74 to TP47, TP75 to TP48, TP76 to TP49, TP77 to TP50, TP78 to TP51, TP43 to TP52, TP44 to TP53, TP45 to TP54, TP46 to TP55, TP47 to TP56, TP48 to TP57, TP49 to TP58, TP50 to TP59, TP51 to TP60, TP79 to TP61, TP80 to TP62, TP81 to TP63, TP82 to TP64, TP83 to TP65, TP84 to TP66, TP85 to TP67, TP86 to TP68, TP87 to TP69, TP52 to TP70, TP53 to TP71, TP54 to TP72, TP55 to TP73, TP56 to TP74, TP57 to TP75, TP58 to TP76, TP59 to TP77, TP60 to TP78, TP88 to TP79, TP89 to TP80, TP90 to TP81, TP91 to TP82, TP92 to TP83, TP93 to TP84, TP94 to TP85, TP95 to TP86, TP96 to TP87, TP61 to TP88, TP62 to TP89, TP63 to TP90, TP64 to TP91, TP65 to TP92, TP66 to TP93, TP67 to TP94, TP68 to TP95, TP69 to TP96
Routing:
- net Net-(T8-AB): track 0.00 -> 152.9 mm, vias 0 -> 2
- net Net-(T1-AB): track 0.00 -> 152.9 mm, vias 0 -> 2
- net Net-(T2-AB): track 0.00 -> 152.9 mm, vias 0 -> 2
- net Net-(T7-AB): track 0.00 -> 152.9 mm, vias 0 -> 2
- net Net-(T6-AB): track 0.00 -> 152.9 mm, vias 0 -> 2
- net Net-(T5-AB): track 0.00 -> 152.9 mm, vias 0 -> 2
- net Net-(T4-AB): track 0.00 -> 152.9 mm, vias 0 -> 2
- net Net-(T3-AB): track 0.00 -> 152.9 mm, vias 0 -> 2
- net Net-(J10-Pad1): track 0.00 -> 143.9 mm
- net Net-(J7-Pad4): track 0.00 -> 143.9 mm
- net Net-(J5-Pad4): track 0.00 -> 143.9 mm
- net Net-(J17-Pad4): track 0.00 -> 143.9 mm
- net Net-(J15-Pad4): track 0.00 -> 143.9 mm
- net Net-(J13-Pad4): track 0.00 -> 143.9 mm
- net Net-(J11-Pad4): track 0.00 -> 143.9 mm
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Other:
- board size 390.2 x 170.1 mm -> 311 x 170.1 mm

Commit message: convert to 4 layer board and add power/gnd planes
Parts:
- moved TP13 59.2 mm to (84.8, 187.4)
- moved TP14 59.2 mm to (89.5, 187.4)
- moved TP15 59.2 mm to (94.1, 187.4)
- moved TP16 59.2 mm to (98.8, 187.4)
- moved TP17 59.2 mm to (103.4, 187.4)
- moved TP18 59.2 mm to (108.1, 187.4)
- moved TP19 59.2 mm to (112.7, 187.4)
- moved TP20 59.2 mm to (117.4, 187.4)
- moved TP21 59.2 mm to (122.0, 187.4)
- moved TP22 59.2 mm to (126.7, 187.4)
- moved TP23 59.2 mm to (131.3, 187.4)
- moved TP24 59.2 mm to (136.0, 187.4)
- moved U7 49.1 mm to (129.2, 160.4)
Connections:
- J10 pad SH: GND -> GNDD
- J12 pad SH: GND -> GNDD
- J14 pad SH: GND -> GNDD
- J16 pad SH: GND -> GNDD
- J18 pad SH: GND -> GNDD
- J4 pad SH: GND -> GNDD
- J6 pad SH: GND -> GNDD
- J8 pad SH: GND -> GNDD
Routing:
- net Net-(J3-Pad1): track 130.9 -> 142.1 mm
- added copper zone on In1.Cu, net +5V
- added copper zone on In1.Cu, net +5VA
- added copper zone on In2.Cu, net GND
- added copper zone on In2.Cu, net GNDD
Other:
- copper layers 2 -> 4

Commit message: fix controlsw/hooksw subsheet error
Connections:
- Q1 pad 2: /LineCtrl1/LineCtrlSingle1/hookSW1 -> /lineCtrls3
- Q10 pad 2: /LineCtrl3/LineCtrlSingle1/controlSW1 -> /lineCtrls9
- Q11 pad 2: /LineCtrl3/LineCtrlSingle2/hookSW1 -> /lineCtrls12
- Q12 pad 2: /LineCtrl3/LineCtrlSingle2/controlSW1 -> /lineCtrls10
- Q13 pad 2: /LineCtrl4/LineCtrlSingle1/hookSW1 -> /lineCtrls15
- Q14 pad 2: /LineCtrl4/LineCtrlSingle1/controlSW1 -> /lineCtrls13
- Q15 pad 2: /LineCtrl4/LineCtrlSingle2/hookSW1 -> /lineCtrls16
- Q16 pad 2: /LineCtrl4/LineCtrlSingle2/controlSW1 -> /lineCtrls14
- Q2 pad 2: /LineCtrl1/LineCtrlSingle1/controlSW1 -> /lineCtrls1
- Q3 pad 2: /LineCtrl1/LineCtrlSingle2/hookSW1 -> /lineCtrls4
- Q4 pad 2: /LineCtrl1/LineCtrlSingle2/controlSW1 -> /lineCtrls2
- Q5 pad 2: /LineCtrl2/LineCtrlSingle1/hookSW1 -> /lineCtrls7
- Q6 pad 2: /LineCtrl2/LineCtrlSingle1/controlSW1 -> /lineCtrls5
- Q7 pad 2: /LineCtrl2/LineCtrlSingle2/hookSW1 -> /lineCtrls8
- Q8 pad 2: /LineCtrl2/LineCtrlSingle2/controlSW1 -> /lineCtrls6
- Q9 pad 2: /LineCtrl3/LineCtrlSingle1/hookSW1 -> /lineCtrls11
- R14 pad 2: /LineCtrl1/LineCtrlSingle1/hookSW1 -> /lineCtrls3
- R16 pad 1: /LineCtrl1/LineCtrlSingle1/controlSW1 -> /lineCtrls1
- R22 pad 2: /LineCtrl1/LineCtrlSingle2/hookSW1 -> /lineCtrls4
- R24 pad 1: /LineCtrl1/LineCtrlSingle2/controlSW1 -> /lineCtrls2
- R30 pad 2: /LineCtrl2/LineCtrlSingle1/hookSW1 -> /lineCtrls7
- R32 pad 1: /LineCtrl2/LineCtrlSingle1/controlSW1 -> /lineCtrls5
- R38 pad 2: /LineCtrl2/LineCtrlSingle2/hookSW1 -> /lineCtrls8
- R40 pad 1: /LineCtrl2/LineCtrlSingle2/controlSW1 -> /lineCtrls6
- R46 pad 2: /LineCtrl3/LineCtrlSingle1/hookSW1 -> /lineCtrls11
- R48 pad 1: /LineCtrl3/LineCtrlSingle1/controlSW1 -> /lineCtrls9
- R54 pad 2: /LineCtrl3/LineCtrlSingle2/hookSW1 -> /lineCtrls12
- R56 pad 1: /LineCtrl3/LineCtrlSingle2/controlSW1 -> /lineCtrls10
- R62 pad 2: /LineCtrl4/LineCtrlSingle1/hookSW1 -> /lineCtrls15
- R64 pad 1: /LineCtrl4/LineCtrlSingle1/controlSW1 -> /lineCtrls13
- R70 pad 2: /LineCtrl4/LineCtrlSingle2/hookSW1 -> /lineCtrls16
- R72 pad 1: /LineCtrl4/LineCtrlSingle2/controlSW1 -> /lineCtrls14
- TP31 pad 1: /LineCtrl1/LineCtrlSingle1/hookSW1 -> /lineCtrls3
- TP32 pad 1: /LineCtrl1/LineCtrlSingle1/controlSW1 -> /lineCtrls1
- TP40 pad 1: /LineCtrl1/LineCtrlSingle2/hookSW1 -> /lineCtrls4
- TP41 pad 1: /LineCtrl1/LineCtrlSingle2/controlSW1 -> /lineCtrls2
- TP49 pad 1: /LineCtrl2/LineCtrlSingle1/hookSW1 -> /lineCtrls7
- TP50 pad 1: /LineCtrl2/LineCtrlSingle1/controlSW1 -> /lineCtrls5
- TP58 pad 1: /LineCtrl2/LineCtrlSingle2/hookSW1 -> /lineCtrls8
- TP59 pad 1: /LineCtrl2/LineCtrlSingle2/controlSW1 -> /lineCtrls6
- TP67 pad 1: /LineCtrl3/LineCtrlSingle1/hookSW1 -> /lineCtrls11
- TP68 pad 1: /LineCtrl3/LineCtrlSingle1/controlSW1 -> /lineCtrls9
- TP76 pad 1: /LineCtrl3/LineCtrlSingle2/hookSW1 -> /lineCtrls12
- TP77 pad 1: /LineCtrl3/LineCtrlSingle2/controlSW1 -> /lineCtrls10
- TP85 pad 1: /LineCtrl4/LineCtrlSingle1/hookSW1 -> /lineCtrls15
- TP86 pad 1: /LineCtrl4/LineCtrlSingle1/controlSW1 -> /lineCtrls13
- TP94 pad 1: /LineCtrl4/LineCtrlSingle2/hookSW1 -> /lineCtrls16
- TP95 pad 1: /LineCtrl4/LineCtrlSingle2/controlSW1 -> /lineCtrls14
Routing:
- net /TransferBtns/shiftLd: track 0.00 -> 370.5 mm, vias 0 -> 1
- net /TransferBtns/shiftInh: track 0.00 -> 363.0 mm
- net /TransferBtns/shiftClk: track 0.00 -> 359.6 mm, vias 0 -> 2
- net /TransferBtns/shiftOut: track 0.00 -> 339.8 mm
- net /ADC/adcCH1: track 0.00 -> 112.8 mm
- net /ADC/adcCH2: track 0.00 -> 105.5 mm
- net /SPI.spi0clk: track 0.00 -> 103.2 mm
- net /SPI.spi0cs0: track 0.00 -> 99.8 mm
- net /ADC/adcCH3: track 0.00 -> 97.9 mm
- net /ADC/adcCH4: track 0.00 -> 95.1 mm
- net /SPI.spi0miso: track 0.00 -> 93.4 mm, vias 0 -> 2
- net /SPI.spi0mosi: track 0.00 -> 92.7 mm, vias 0 -> 2
- net /ADC/adcCH5: track 0.00 -> 87.9 mm
- net /ADC/adcCH8: track 0.00 -> 86.8 mm
- net /ADC/adcCH6: track 0.00 -> 86.2 mm
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Other:
- board text added: "1"
- board text added: "2"
- board text added: "3"
- board text added: "4"
- board text added: "5"
- board text added: "6"
- board text added: "7"
- board text added: "8"
- board text added: "ADC"
- board text added: "ADC Channels"
- board text added: "LM358 Dual Opamps"
- board text added: "M5 PBX Sniffer V2"
- board text added: "MCP3008 10-bit 8-Channel ADC"
- board text added: "Made with love by Tobe Cynar This device handles the automatic transferring of calls and extracts the audio data off the phone lines during the M5 Telethon"
- board text added: "Opamps"
- board text added: "Pull-up Resistors"
- board text added: "SPI"
- board text added: "clk"
- board text added: "cs"
- board text added: "miso"
- board text added: "mosi"
