File: pbx-sniffer-v2.kicad_pcb (KiCad board)
At the start: 4 copper layers, 321 x 170.1 mm, 301 parts, among them J1 8P8C, J10 6P4C, J11 6P4C, J12 6P4C, J13 6P4C, J14 6P4C, J15 6P4C, J16 6P4C, J17 6P4C, J18 6P4C, J2 8P8C, J3 6P4C, J4 6P4C, J5 6P4C, J6 6P4C, J7 6P4C, J8 6P4C, J9 6P4C, K1 Relay_SPST-NO, K10 Relay_SPDT, K11 Relay_SPST-NO, K12 Relay_SPDT, K13 Relay_SPST-NO, K14 Relay_SPDT, K15 Relay_SPST-NO, K16 Relay_SPDT, K2 Relay_SPDT, K3 Relay_SPST-NO, K4 Relay_SPDT, K5 Relay_SPST-NO, K6 Relay_SPDT, K7 Relay_SPST-NO, K8 Relay_SPDT, K9 Relay_SPST-NO, Q1 PMOS, Q10 PMOS, Q11 PMOS, Q12 PMOS, Q13 PMOS, Q14 PMOS, Q15 PMOS, Q16 PMOS, Q2 PMOS, Q3 PMOS, Q4 PMOS, Q5 PMOS, Q6 PMOS, Q7 PMOS, Q8 PMOS, Q9 PMOS, T1 Transformer_1P_1S, T2 Transformer_1P_1S, T3 Transformer_1P_1S, T4 Transformer_1P_1S, T5 Transformer_1P_1S, T6 Transformer_1P_1S, T7 Transformer_1P_1S, T8 Transformer_1P_1S, U1 STM32NucleoF303RE, U2 LM358, U3 LM358, U4 LM358, U5 LM358, U6 74LS165, U7 MCP3008

Commit message: added power mux, finished up schematic and picking footprints/partnumbers
Parts:
- removed C1, C10, C11, C12, C13, C14, C15, C16, C17, C18, C19, C2, C20, C21, C22, C23, C24, C3, C4, C5, C6, C7, C8, C9: 0.47u, Capacitor_THT:C_Rect_L7.0mm_W2.0mm_P5.00mm
- removed D1, D10, D11, D12, D13, D14, D15, D16, D17, D18, D19, D2, D20, D21, D22, D23, D24, D25, D26, D27, D28, D29, D3, D30, D31, D32, D4, D5, D6, D7, D8, D9: 1N4148, Diode_THT:D_DO-35_SOD27_P7.62mm_Horizontal
- removed H1 (x4): MountingHole_5.3mm_M5_DIN965_Pad, MountingHole:MountingHole_5.3mm_M5_DIN965_Pad
- removed J1, J2: 8P8C, Phones:AMPHENOL_54602-908LF
- removed J10, J11, J12, J13, J14, J15, J16, J17, J18, J3, J4, J5, J6, J7, J8, J9: 6P4C, Phones:CUI_CRJ050-1-TH
- removed JP1, JP2, JP3, JP4, JP5, JP6, JP7, JP8: Jumper_1-2, Jumper:SolderJumper-3_P1.3mm_Bridged2Bar12_RoundedPad1.0x1.5mm
- removed K1, K11, K13, K15, K3, K5, K7, K9: Relay_SPST-NO, Relay_THT:Relay_SPST_StandexMeder_SIL_Form1A
- removed K10, K12, K14, K16, K2, K4, K6, K8: Relay_SPDT, Phones:K_AZ943-1C_AMZ
- removed Q1, Q10, Q11, Q12, Q13, Q14, Q15, Q16, Q2, Q3, Q4, Q5, Q6, Q7, Q8, Q9: PMOS, Package_TO_SOT_THT:TO-92_HandSolder
- removed R1, R10, R11, R13, R14, R16, R17, R18, R19, R2, R21, R22, R24, R25, R26, R27, R29, R3, R30, R32, R33, R34, R35, R37, R38, R4, R40, R41, R42, R43, R45, R46, R48, R49, R5, R50, R51, R53, R54, R56, R57, R58, R59, R6, R61, R62, R64, R65, R66, R67, R69, R7, R70, R72, R8, R9: 10k, Resistor_THT:R_Axial_DIN0207_L6.3mm_D2.5mm_P7.62mm_Horizontal
- removed R12, R20, R28, R36, R44, R52, R60, R68: 1k, Resistor_THT:R_Axial_DIN0207_L6.3mm_D2.5mm_P7.62mm_Horizontal
- removed R15, R23, R31, R39, R47, R55, R63, R71: 500, Resistor_THT:R_Axial_DIN0207_L6.3mm_D2.5mm_P7.62mm_Horizontal
- removed T1, T2, T3, T4, T5, T6, T7, T8: Transformer_1P_1S, Phones:TY-145P
- removed TP1, TP10, TP11, TP12, TP13, TP14, TP15, TP16, TP17, TP18, TP19, TP2, TP20, TP21, TP22, TP23, TP24, TP25, TP26, TP27, TP28, TP29, TP3, TP30, TP31, TP32, TP33, TP34, TP35, TP36, TP37, TP38, TP39, TP4, TP40, TP41, TP42, TP43, TP44, TP45, TP46, TP47, TP48, TP49, TP5, TP50, TP51, TP52, TP53, TP54, TP55, TP56, TP57, TP58, TP59, TP6, TP60, TP61, TP62, TP63, TP64, TP65, TP66, TP67, TP68, TP69, TP7, TP70, TP71, TP72, TP73, TP74, TP75, TP76, TP77, TP78, TP79, TP8, TP80, TP81, TP82, TP83, TP84, TP85, TP86, TP87, TP88, TP89, TP9, TP90, TP91, TP92, TP93, TP94, TP95, TP96: TestPoint, Testpoints:M5_3in1_TestPoint
- removed U1: STM32NucleoF303RE, Nucleo:STM32NucleoF303RE
- removed U2, U3, U4, U5: LM358, Package_DIP:DIP-8_W7.62mm
- removed U6: 74LS165, Package_DIP:DIP-16_W7.62mm
- removed U7: MCP3008, Package_DIP:DIP-16_W7.62mm
Routing:
- net /lineCtrls16: track 374.9 -> 0.00 mm, vias 3 -> 0
- net /TransferBtns/shiftLd: track 371.3 -> 0.00 mm, vias 2 -> 0
- net /TransferBtns/shiftInh: track 363.1 -> 0.00 mm, vias 1 -> 0
- net /TransferBtns/shiftClk: track 359.6 -> 0.00 mm, vias 3 -> 0
- net /TransferBtns/shiftOut: track 339.8 -> 0.00 mm, vias 1 -> 0
- net /lineCtrls14: track 337.3 -> 0.00 mm, vias 1 -> 0
- net /LineCtrl4/LineCtrlSingle2/ampV+: track 327.1 -> 0.00 mm, vias 1 -> 0
- net /lineCtrls13: track 302.7 -> 0.00 mm, vias 1 -> 0
- net /ADC/adcCH8: track 300.4 -> 0.00 mm
- net /ADC/adcCH7: track 273.4 -> 0.00 mm
- net /lineCtrls10: track 264.6 -> 0.00 mm, vias 1 -> 0
- net /LineCtrl4/LineCtrlSingle1/ampV+: track 260.9 -> 0.00 mm, vias 3 -> 0
- net /lineCtrls15: track 251.4 -> 0.00 mm, vias 2 -> 0
- net /ADC/adcCH6: track 247.4 -> 0.00 mm, vias 1 -> 0
- net /ADC/adcCH5: track 238.0 -> 0.00 mm
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- removed copper zone on In1.Cu, net +5V
- removed copper zone on In1.Cu, net +5VA
- removed copper zone on In2.Cu, net GND
- removed copper zone on In2.Cu, net GNDD
Other:
- board outline removed
- board text removed: "1"
- board text removed: "2"
- board text removed: "3"
- board text removed: "4"
- board text removed: "5"
- board text removed: "6"
- board text removed: "7"
- board text removed: "74LS165 Shift Register"
- board text removed: "8"
- board text removed: "ADC"
- board text removed: "ADC Channels"
- board text removed: "LM358 Dual Opamps"
- board text removed: "M5 PBX Sniffer V2"
- board text removed: "MCP3008 10-bit 8-Channel ADC"
- board text removed: "Made with love by Tobe Cynar This device handles the automatic transferring of calls and extracts the audio data off the phone lines during the M5 Telethon"
- board text removed: "Opamps"
- board text removed: "Pull-up Resistors"
- board text removed: "SPI"
- board text removed: "Transfer Btns"
- board text removed: "clk"
- board text removed: "cs"
- board text removed: "inh"
- board text removed: "ld"
- board text removed: "miso"
- board text removed: "mosi"
- board text removed: "out"

Commit message: nearly complete layout lol
Parts:
- added C1: 100n, Capacitor_SMD:C_0805_2012Metric, B.Cu at (199.9, 178.9)
- added C10: 100n, Capacitor_SMD:C_0805_2012Metric, B.Cu at (205.9, 182.6)
- added C11: 100n, Capacitor_SMD:C_0805_2012Metric, B.Cu at (208.9, 182.6)
- added C12: 100n, Capacitor_SMD:C_0805_2012Metric, B.Cu at (199.9, 186.2)
- added C13: 100n, Capacitor_SMD:C_0805_2012Metric, B.Cu at (202.9, 186.2)
- added C14: 100n, Capacitor_SMD:C_0805_2012Metric, B.Cu at (205.9, 186.2)
- added C15: 4.7u, Capacitor_SMD:C_0805_2012Metric, B.Cu at (208.9, 186.2)
- added C16: 10n, Capacitor_SMD:C_0805_2012Metric, B.Cu at (195.2, 179.0)
- added C17: 1u, Capacitor_SMD:C_0805_2012Metric, B.Cu at (195.2, 182.0)
- added C18: 100n, Capacitor_SMD:C_0805_2012Metric, F.Cu at (223.1, 127.0)
- added C19: 0.47u, Capacitor_SMD:C_0805_2012Metric, F.Cu at (231.8, 139.6)
- added C2: 100n, Capacitor_SMD:C_0805_2012Metric, B.Cu at (202.9, 178.9)
- added C20: 0.47u, Capacitor_SMD:C_0805_2012Metric, F.Cu at (236.0, 160.1)
- added C21: 1u, Capacitor_SMD:C_0805_2012Metric, F.Cu at (222.2, 140.0)
- added C22: 0.47u, Capacitor_SMD:C_0805_2012Metric, F.Cu at (264.9, 139.6)
- added C23: 0.47u, Capacitor_SMD:C_0805_2012Metric, F.Cu at (269.1, 160.1)
- added C24: 1u, Capacitor_SMD:C_0805_2012Metric, F.Cu at (255.3, 140.0)
- added C25: 100n, Capacitor_SMD:C_0805_2012Metric, F.Cu at (289.2, 127.0)
- added C26: 0.47u, Capacitor_SMD:C_0805_2012Metric, F.Cu at (298.0, 139.6)
- added C27: 0.47u, Capacitor_SMD:C_0805_2012Metric, F.Cu at (302.2, 160.1)
- added C28: 1u, Capacitor_SMD:C_0805_2012Metric, F.Cu at (288.4, 140.0)
- added C29: 0.47u, Capacitor_SMD:C_0805_2012Metric, F.Cu at (331.1, 139.6)
- added C3: 100n, Capacitor_SMD:C_0805_2012Metric, B.Cu at (205.9, 178.9)
- added C30: 0.47u, Capacitor_SMD:C_0805_2012Metric, F.Cu at (335.3, 160.1)
- added C31: 1u, Capacitor_SMD:C_0805_2012Metric, F.Cu at (321.5, 140.0)
- added C32: 100n, Capacitor_SMD:C_0805_2012Metric, F.Cu at (355.6, 127.2)
- added C33: 0.47u, Capacitor_SMD:C_0805_2012Metric, F.Cu at (364.3, 139.6)
- added C34: 0.47u, Capacitor_SMD:C_0805_2012Metric, F.Cu at (368.5, 160.1)
- added C35: 1u, Capacitor_SMD:C_0805_2012Metric, F.Cu at (354.7, 140.0)
- added C36: 0.47u, Capacitor_SMD:C_0805_2012Metric, F.Cu at (397.4, 139.6)
- added C37: 0.47u, Capacitor_SMD:C_0805_2012Metric, F.Cu at (401.6, 160.1)
- added C38: 1u, Capacitor_SMD:C_0805_2012Metric, F.Cu at (387.8, 140.0)
- added C39: 100n, Capacitor_SMD:C_0805_2012Metric, F.Cu at (421.6, 127.0)
- added C4: 100n, Capacitor_SMD:C_0805_2012Metric, F.Cu at (174.2, 176.3)
- added C40: 0.47u, Capacitor_SMD:C_0805_2012Metric, F.Cu at (430.5, 139.6)
- added C41: 0.47u, Capacitor_SMD:C_0805_2012Metric, F.Cu at (434.7, 160.1)
- added C42: 1u, Capacitor_SMD:C_0805_2012Metric, F.Cu at (420.9, 140.0)
- added C43: 0.47u, Capacitor_SMD:C_0805_2012Metric, F.Cu at (463.6, 139.6)
- added C44: 0.47u, Capacitor_SMD:C_0805_2012Metric, F.Cu at (467.8, 160.1)
- added C45: 1u, Capacitor_SMD:C_0805_2012Metric, F.Cu at (454.0, 140.0)
- added C5: 100n, Capacitor_SMD:C_0805_2012Metric, B.Cu at (208.9, 178.9)
- added C6: 100n, Capacitor_SMD:C_0805_2012Metric, B.Cu at (199.9, 182.6)
- added C7: 22p, Capacitor_SMD:C_0805_2012Metric, F.Cu at (195.1, 172.5)
- added C8: 22p, Capacitor_SMD:C_0805_2012Metric, F.Cu at (195.1, 175.5)
- added C9: 100n, Capacitor_SMD:C_0805_2012Metric, B.Cu at (202.9, 182.6)
- added D1: LED, Resistor_SMD:R_0603_1608Metric, F.Cu at (179.2, 187.6)
- added D10: M7, Diode_SMD:D_SMA, F.Cu at (275.5, 165.6)
- added D11: LED, Resistor_SMD:R_0603_1608Metric, F.Cu at (275.5, 176.0)
- added D12: LED, Resistor_SMD:R_0603_1608Metric, F.Cu at (275.5, 178.4)
- added D13: M7, Diode_SMD:D_SMA, F.Cu at (277.1, 185.4)
- added D14: RB520S30T5G, Diode_SMD:D_SOD-523, F.Cu at (298.4, 159.0)
- added D15: RB520S30T5G, Diode_SMD:D_SOD-523, F.Cu at (306.0, 159.0)
- added D16: M7, Diode_SMD:D_SMA, F.Cu at (308.6, 165.6)
- added D17: LED, Resistor_SMD:R_0603_1608Metric, F.Cu at (308.7, 176.0)
- added D18: LED, Resistor_SMD:R_0603_1608Metric, F.Cu at (308.7, 178.4)
- added D19: M7, Diode_SMD:D_SMA, F.Cu at (310.2, 185.4)
- added D2: RB520S30T5G, Diode_SMD:D_SOD-523, F.Cu at (232.2, 159.0)
- added D20: RB520S30T5G, Diode_SMD:D_SOD-523, F.Cu at (331.5, 159.0)
- added D21: RB520S30T5G, Diode_SMD:D_SOD-523, F.Cu at (339.1, 159.0)
- added D22: M7, Diode_SMD:D_SMA, F.Cu at (341.7, 165.6)
- added D23: LED, Resistor_SMD:R_0603_1608Metric, F.Cu at (341.8, 176.0)
- added D24: LED, Resistor_SMD:R_0603_1608Metric, F.Cu at (341.8, 178.4)
- added D25: M7, Diode_SMD:D_SMA, F.Cu at (343.3, 185.4)
- added D26: RB520S30T5G, Diode_SMD:D_SOD-523, F.Cu at (364.7, 159.0)
- added D27: RB520S30T5G, Diode_SMD:D_SOD-523, F.Cu at (372.3, 159.0)
- added D28: M7, Diode_SMD:D_SMA, F.Cu at (374.9, 165.6)
- added D29: LED, Resistor_SMD:R_0603_1608Metric, F.Cu at (374.9, 176.0)
- added D3: RB520S30T5G, Diode_SMD:D_SOD-523, F.Cu at (239.8, 159.0)
- added D30: LED, Resistor_SMD:R_0603_1608Metric, F.Cu at (374.9, 178.4)
- added D31: M7, Diode_SMD:D_SMA, F.Cu at (376.5, 185.4)
- added D32: RB520S30T5G, Diode_SMD:D_SOD-523, F.Cu at (397.8, 159.0)
- added D33: RB520S30T5G, Diode_SMD:D_SOD-523, F.Cu at (405.4, 159.0)
- added D34: M7, Diode_SMD:D_SMA, F.Cu at (408.0, 165.6)
- added D35: LED, Resistor_SMD:R_0603_1608Metric, F.Cu at (408.0, 176.0)
- added D36: LED, Resistor_SMD:R_0603_1608Metric, F.Cu at (408.0, 178.4)
- added D37: M7, Diode_SMD:D_SMA, F.Cu at (409.6, 185.4)
- added D38: RB520S30T5G, Diode_SMD:D_SOD-523, F.Cu at (430.9, 159.0)
- added D39: RB520S30T5G, Diode_SMD:D_SOD-523, F.Cu at (438.5, 159.0)
- added D4: M7, Diode_SMD:D_SMA, F.Cu at (242.4, 165.6)
- added D40: M7, Diode_SMD:D_SMA, F.Cu at (441.1, 165.6)
- added D41: LED, Resistor_SMD:R_0603_1608Metric, F.Cu at (441.1, 176.0)
- added D42: LED, Resistor_SMD:R_0603_1608Metric, F.Cu at (441.1, 178.4)
- added D43: M7, Diode_SMD:D_SMA, F.Cu at (442.7, 185.4)
- added D44: RB520S30T5G, Diode_SMD:D_SOD-523, F.Cu at (464.0, 159.0)
- added D45: RB520S30T5G, Diode_SMD:D_SOD-523, F.Cu at (471.6, 159.0)
- added D46: M7, Diode_SMD:D_SMA, F.Cu at (474.2, 165.6)
- added D47: LED, Resistor_SMD:R_0603_1608Metric, F.Cu at (474.2, 176.0)
- added D48: LED, Resistor_SMD:R_0603_1608Metric, F.Cu at (474.2, 178.4)
- added D49: M7, Diode_SMD:D_SMA, F.Cu at (475.8, 185.4)
- added D5: LED, Resistor_SMD:R_0603_1608Metric, F.Cu at (242.4, 176.0)
- added D50: LED, Resistor_SMD:R_0603_1608Metric, F.Cu at (500.8, 171.2)
- added D51: LED, Resistor_SMD:R_0603_1608Metric, F.Cu at (500.8, 174.2)
- added D52: LED, Resistor_SMD:R_0603_1608Metric, F.Cu at (500.8, 177.1)
- added D53: LED, Resistor_SMD:R_0603_1608Metric, F.Cu at (500.8, 180.0)
- added D54: LED, Resistor_SMD:R_0603_1608Metric, F.Cu at (500.8, 183.0)
- added D55: LED, Resistor_SMD:R_0603_1608Metric, F.Cu at (500.8, 185.9)
- added D56: LED, Resistor_SMD:R_0603_1608Metric, F.Cu at (500.8, 188.9)
- added D57: LED, Resistor_SMD:R_0603_1608Metric, F.Cu at (500.8, 191.8)
- added D6: LED, Resistor_SMD:R_0603_1608Metric, F.Cu at (242.4, 178.4)
- added D7: M7, Diode_SMD:D_SMA, F.Cu at (244.0, 185.4)
- added D8: RB520S30T5G, Diode_SMD:D_SOD-523, F.Cu at (265.3, 159.0)
- added D9: RB520S30T5G, Diode_SMD:D_SOD-523, F.Cu at (272.9, 159.0)
- added FB1: FerriteBead_Small, Inductor_SMD:L_0805_2012Metric, F.Cu at (193.5, 192.6)
- added FB2: FerriteBead_Small, Inductor_SMD:L_0805_2012Metric, F.Cu at (193.5, 189.6)
- added H1: MountingHole, MountingHole:MountingHole_5.3mm_M5_Pad, F.Cu at (205.0, 115.4)
- added H2: MountingHole, MountingHole:MountingHole_5.3mm_M5_Pad, F.Cu at (503.0, 115.4)
- added H3: MountingHole, MountingHole:MountingHole_5.3mm_M5_Pad, F.Cu at (154.0, 201.4)
- added H4: MountingHole, MountingHole:MountingHole_5.3mm_M5_Pad, F.Cu at (503.0, 201.4)
- added J1: Conn_01x02_Socket, TerminalBlock_CUI:TerminalBlock_CUI_TB007-508-02_1x02_P5.08mm_Horizontal, F.Cu at (189.2, 203.2)
- added J10: 6P4C, Phones:CUI_CRJ050-1-TH, F.Cu at (302.2, 202.2)
- added J11: 6P4C, Phones:CUI_CRJ050-1-TH, F.Cu at (335.3, 114.8)
- added J12: 6P4C, Phones:CUI_CRJ050-1-TH, F.Cu at (335.3, 202.2)
- added J13: 6P4C, Phones:CUI_CRJ050-1-TH, F.Cu at (368.5, 114.8)
- added J14: 6P4C, Phones:CUI_CRJ050-1-TH, F.Cu at (368.5, 202.2)
- added J15: 6P4C, Phones:CUI_CRJ050-1-TH, F.Cu at (401.6, 114.8)
- added J16: 6P4C, Phones:CUI_CRJ050-1-TH, F.Cu at (401.6, 202.2)
- added J17: 6P4C, Phones:CUI_CRJ050-1-TH, F.Cu at (434.7, 114.8)
- added J18: 6P4C, Phones:CUI_CRJ050-1-TH, F.Cu at (434.7, 202.2)
- added J19: 6P4C, Phones:CUI_CRJ050-1-TH, F.Cu at (467.8, 114.8)
- added J2: USB_C_Receptacle_USB2.0_14P, Connector_USB:USB_C_Receptacle_Amphenol_12401610E4-2A, F.Cu at (172.2, 203.2)
- added J20: 6P4C, Phones:CUI_CRJ050-1-TH, F.Cu at (467.8, 202.2)
- added J21: 8P8C, Phones:AMPHENOL_54602-908LF, F.Cu at (504.2, 136.2)
- added J22: 8P8C, Phones:AMPHENOL_54602-908LF, F.Cu at (504.2, 152.3)
- added J3: Conn_01x04_Socket, Connector_PinHeader_2.54mm:PinHeader_1x04_P2.54mm_Vertical, F.Cu at (155.5, 163.1)
- added J4: Conn_01x03_Socket, Connector_PinHeader_2.54mm:PinHeader_1x03_P2.54mm_Vertical, F.Cu at (164.6, 163.1)
- added J5: 6P4C, Phones:CUI_CRJ050-1-TH, F.Cu at (236.0, 114.8)
- added J6: 6P4C, Phones:CUI_CRJ050-1-TH, F.Cu at (236.0, 202.2)
- added J7: 6P4C, Phones:CUI_CRJ050-1-TH, F.Cu at (269.1, 114.8)
- added J8: 6P4C, Phones:CUI_CRJ050-1-TH, F.Cu at (269.1, 202.2)
- added J9: 6P4C, Phones:CUI_CRJ050-1-TH, F.Cu at (302.2, 114.8)
- added JP1: Jumper_1-2, Jumper:SolderJumper-3_P1.3mm_Bridged2Bar12_RoundedPad1.0x1.5mm, F.Cu at (243.0, 140.3)
- added JP2: Jumper_1-2, Jumper:SolderJumper-3_P1.3mm_Bridged2Bar12_RoundedPad1.0x1.5mm, F.Cu at (276.1, 140.3)
- added JP3: Jumper_1-2, Jumper:SolderJumper-3_P1.3mm_Bridged2Bar12_RoundedPad1.0x1.5mm, F.Cu at (309.2, 140.3)
- added JP4: Jumper_1-2, Jumper:SolderJumper-3_P1.3mm_Bridged2Bar12_RoundedPad1.0x1.5mm, F.Cu at (342.3, 140.3)
- added JP5: Jumper_1-2, Jumper:SolderJumper-3_P1.3mm_Bridged2Bar12_RoundedPad1.0x1.5mm, F.Cu at (375.5, 140.3)
- added JP6: Jumper_1-2, Jumper:SolderJumper-3_P1.3mm_Bridged2Bar12_RoundedPad1.0x1.5mm, F.Cu at (408.6, 140.3)
- added JP7: Jumper_1-2, Jumper:SolderJumper-3_P1.3mm_Bridged2Bar12_RoundedPad1.0x1.5mm, F.Cu at (441.7, 140.3)
- added JP8: Jumper_1-2, Jumper:SolderJumper-3_P1.3mm_Bridged2Bar12_RoundedPad1.0x1.5mm, F.Cu at (474.8, 140.3)
- added K1: Relay_SPST-NO, Relay_SMD:Relay_2P2T_10x6mm_TE_IMxxG, F.Cu at (234.8, 172.6)
- added K10: Relay_SPDT, Relay_SMD:Relay_2P2T_10x6mm_TE_IMxxG, F.Cu at (367.3, 181.8)
- added K11: Relay_SPST-NO, Relay_SMD:Relay_2P2T_10x6mm_TE_IMxxG, F.Cu at (400.4, 172.6)
- added K12: Relay_SPDT, Relay_SMD:Relay_2P2T_10x6mm_TE_IMxxG, F.Cu at (400.4, 181.8)
- added K13: Relay_SPST-NO, Relay_SMD:Relay_2P2T_10x6mm_TE_IMxxG, F.Cu at (433.5, 172.6)
- added K14: Relay_SPDT, Relay_SMD:Relay_2P2T_10x6mm_TE_IMxxG, F.Cu at (433.5, 181.8)
- added K15: Relay_SPST-NO, Relay_SMD:Relay_2P2T_10x6mm_TE_IMxxG, F.Cu at (466.6, 172.6)
- added K16: Relay_SPDT, Relay_SMD:Relay_2P2T_10x6mm_TE_IMxxG, F.Cu at (466.6, 181.8)
- added K2: Relay_SPDT, Relay_SMD:Relay_2P2T_10x6mm_TE_IMxxG, F.Cu at (234.8, 181.8)
- added K3: Relay_SPST-NO, Relay_SMD:Relay_2P2T_10x6mm_TE_IMxxG, F.Cu at (267.9, 172.6)
- added K4: Relay_SPDT, Relay_SMD:Relay_2P2T_10x6mm_TE_IMxxG, F.Cu at (267.9, 181.8)
- added K5: Relay_SPST-NO, Relay_SMD:Relay_2P2T_10x6mm_TE_IMxxG, F.Cu at (301.0, 172.6)
- added K6: Relay_SPDT, Relay_SMD:Relay_2P2T_10x6mm_TE_IMxxG, F.Cu at (301.0, 181.8)
- added K7: Relay_SPST-NO, Relay_SMD:Relay_2P2T_10x6mm_TE_IMxxG, F.Cu at (334.1, 172.6)
- added K8: Relay_SPDT, Relay_SMD:Relay_2P2T_10x6mm_TE_IMxxG, F.Cu at (334.1, 181.8)
- added K9: Relay_SPST-NO, Relay_SMD:Relay_2P2T_10x6mm_TE_IMxxG, F.Cu at (367.3, 172.6)
- added Q1: PMOS, Package_TO_SOT_SMD:SOT-23, F.Cu at (173.1, 191.4)
- added Q10: PMOS, Package_TO_SOT_SMD:SOT-23, F.Cu at (368.5, 164.8)
- added Q11: PMOS, Package_TO_SOT_SMD:SOT-23, F.Cu at (360.3, 187.8)
- added Q12: PMOS, Package_TO_SOT_SMD:SOT-23, F.Cu at (401.6, 164.8)
- added Q13: PMOS, Package_TO_SOT_SMD:SOT-23, F.Cu at (393.4, 187.8)
- added Q14: PMOS, Package_TO_SOT_SMD:SOT-23, F.Cu at (434.7, 164.8)
- added Q15: PMOS, Package_TO_SOT_SMD:SOT-23, F.Cu at (426.5, 187.8)
- added Q16: PMOS, Package_TO_SOT_SMD:SOT-23, F.Cu at (467.9, 164.8)
- added Q17: PMOS, Package_TO_SOT_SMD:SOT-23, F.Cu at (459.6, 187.8)
- added Q2: PMOS, Package_TO_SOT_SMD:SOT-23, F.Cu at (236.1, 164.8)
- added Q3: PMOS, Package_TO_SOT_SMD:SOT-23, F.Cu at (227.8, 187.8)
- added Q4: PMOS, Package_TO_SOT_SMD:SOT-23, F.Cu at (269.2, 164.8)
- added Q5: PMOS, Package_TO_SOT_SMD:SOT-23, F.Cu at (260.9, 187.8)
- added Q6: PMOS, Package_TO_SOT_SMD:SOT-23, F.Cu at (302.3, 164.8)
- added Q7: PMOS, Package_TO_SOT_SMD:SOT-23, F.Cu at (294.0, 187.8)
- added Q8: PMOS, Package_TO_SOT_SMD:SOT-23, F.Cu at (335.4, 164.8)
- added Q9: PMOS, Package_TO_SOT_SMD:SOT-23, F.Cu at (327.1, 187.8)
- added R1: 10k, Resistor_SMD:R_0805_2012Metric, F.Cu at (179.3, 179.6)
- added R10: 1k, Resistor_SMD:R_0805_2012Metric, F.Cu at (222.2, 138.0)
- added R100: 330, Resistor_SMD:R_0805_2012Metric, F.Cu at (496.5, 186.0)
- added R101: 330, Resistor_SMD:R_0805_2012Metric, F.Cu at (496.5, 188.8)
- added R102: 330, Resistor_SMD:R_0805_2012Metric, F.Cu at (496.5, 191.8)
- added R11: 10k, Resistor_SMD:R_0805_2012Metric, F.Cu at (225.7, 138.0)
- added R12: 10k, Resistor_SMD:R_0805_2012Metric, F.Cu at (232.0, 164.6)
- added R13: 600, Resistor_SMD:R_0805_2012Metric, F.Cu at (238.2, 139.6)
- added R14: 330, Resistor_SMD:R_0805_2012Metric, F.Cu at (242.3, 169.8)
- added R15: 10k, Resistor_SMD:R_0805_2012Metric, F.Cu at (227.6, 170.2)
- added R16: 330, Resistor_SMD:R_0805_2012Metric, F.Cu at (242.3, 172.0)
- added R17: 10k, Resistor_SMD:R_0805_2012Metric, F.Cu at (267.1, 139.6)
- added R18: 10k, Resistor_SMD:R_0805_2012Metric, F.Cu at (265.2, 161.2)
- added R19: 10k, Resistor_SMD:R_0805_2012Metric, F.Cu at (272.8, 161.4)
- added R2: 330, Resistor_SMD:R_0805_2012Metric, F.Cu at (179.3, 183.0)
- added R20: 1k, Resistor_SMD:R_0805_2012Metric, F.Cu at (255.3, 138.0)
- added R21: 10k, Resistor_SMD:R_0805_2012Metric, F.Cu at (258.8, 138.0)
- added R22: 10k, Resistor_SMD:R_0805_2012Metric, F.Cu at (265.1, 164.6)
- added R23: 600, Resistor_SMD:R_0805_2012Metric, F.Cu at (271.3, 139.6)
- added R24: 330, Resistor_SMD:R_0805_2012Metric, F.Cu at (275.4, 169.8)
- added R25: 10k, Resistor_SMD:R_0805_2012Metric, F.Cu at (260.7, 170.2)
- added R26: 330, Resistor_SMD:R_0805_2012Metric, F.Cu at (275.4, 172.0)
- added R27: 10k, Resistor_SMD:R_0805_2012Metric, F.Cu at (300.2, 139.6)
- added R28: 10k, Resistor_SMD:R_0805_2012Metric, F.Cu at (298.3, 161.2)
- added R29: 10k, Resistor_SMD:R_0805_2012Metric, F.Cu at (305.9, 161.4)
- added R3: 5.1k, Resistor_SMD:R_0805_2012Metric, F.Cu at (168.5, 191.1)
- added R30: 1k, Resistor_SMD:R_0805_2012Metric, F.Cu at (288.4, 138.0)
- added R31: 10k, Resistor_SMD:R_0805_2012Metric, F.Cu at (291.9, 138.0)
- added R32: 10k, Resistor_SMD:R_0805_2012Metric, F.Cu at (298.2, 164.6)
- added R33: 600, Resistor_SMD:R_0805_2012Metric, F.Cu at (304.4, 139.6)
- added R34: 330, Resistor_SMD:R_0805_2012Metric, F.Cu at (308.5, 169.8)
- added R35: 10k, Resistor_SMD:R_0805_2012Metric, F.Cu at (293.8, 170.2)
- added R36: 330, Resistor_SMD:R_0805_2012Metric, F.Cu at (308.5, 172.0)
- added R37: 10k, Resistor_SMD:R_0805_2012Metric, F.Cu at (333.3, 139.6)
- added R38: 10k, Resistor_SMD:R_0805_2012Metric, F.Cu at (331.5, 161.2)
- added R39: 10k, Resistor_SMD:R_0805_2012Metric, F.Cu at (339.1, 161.4)
- added R4: 5.1k, Resistor_SMD:R_0805_2012Metric, F.Cu at (168.5, 194.4)
- added R40: 1k, Resistor_SMD:R_0805_2012Metric, F.Cu at (321.5, 138.0)
- added R41: 10k, Resistor_SMD:R_0805_2012Metric, F.Cu at (325.0, 138.0)
- added R42: 10k, Resistor_SMD:R_0805_2012Metric, F.Cu at (331.3, 164.6)
- added R43: 600, Resistor_SMD:R_0805_2012Metric, F.Cu at (337.5, 139.6)
- added R44: 330, Resistor_SMD:R_0805_2012Metric, F.Cu at (341.6, 169.8)
- added R45: 10k, Resistor_SMD:R_0805_2012Metric, F.Cu at (326.9, 170.2)
- added R46: 330, Resistor_SMD:R_0805_2012Metric, F.Cu at (341.6, 172.0)
- added R47: 10k, Resistor_SMD:R_0805_2012Metric, F.Cu at (366.5, 139.6)
- added R48: 10k, Resistor_SMD:R_0805_2012Metric, F.Cu at (364.6, 161.2)
- added R49: 10k, Resistor_SMD:R_0805_2012Metric, F.Cu at (372.2, 161.4)
- added R5: 10k, Resistor_SMD:R_0805_2012Metric, F.Cu at (199.1, 198.6)
- added R50: 1k, Resistor_SMD:R_0805_2012Metric, F.Cu at (354.7, 138.0)
- added R51: 10k, Resistor_SMD:R_0805_2012Metric, F.Cu at (358.1, 138.0)
- added R52: 10k, Resistor_SMD:R_0805_2012Metric, F.Cu at (364.5, 164.6)
- added R53: 600, Resistor_SMD:R_0805_2012Metric, F.Cu at (370.7, 139.6)
- added R54: 330, Resistor_SMD:R_0805_2012Metric, F.Cu at (374.7, 169.8)
- added R55: 10k, Resistor_SMD:R_0805_2012Metric, F.Cu at (360.1, 170.2)
- added R56: 330, Resistor_SMD:R_0805_2012Metric, F.Cu at (374.7, 172.0)
- added R57: 10k, Resistor_SMD:R_0805_2012Metric, F.Cu at (399.6, 139.6)
- added R58: 10k, Resistor_SMD:R_0805_2012Metric, F.Cu at (397.7, 161.2)
- added R59: 10k, Resistor_SMD:R_0805_2012Metric, F.Cu at (405.3, 161.4)
- added R6: 390, Resistor_SMD:R_0805_2012Metric, F.Cu at (191.7, 172.5)
- added R60: 1k, Resistor_SMD:R_0805_2012Metric, F.Cu at (387.8, 138.0)
- added R61: 10k, Resistor_SMD:R_0805_2012Metric, F.Cu at (391.3, 138.0)
- added R62: 10k, Resistor_SMD:R_0805_2012Metric, F.Cu at (397.6, 164.6)
- added R63: 600, Resistor_SMD:R_0805_2012Metric, F.Cu at (403.8, 139.6)
- added R64: 330, Resistor_SMD:R_0805_2012Metric, F.Cu at (407.9, 169.8)
- added R65: 10k, Resistor_SMD:R_0805_2012Metric, F.Cu at (393.2, 170.2)
- added R66: 330, Resistor_SMD:R_0805_2012Metric, F.Cu at (407.9, 172.0)
- added R67: 10k, Resistor_SMD:R_0805_2012Metric, F.Cu at (432.7, 139.6)
- added R68: 10k, Resistor_SMD:R_0805_2012Metric, F.Cu at (430.8, 161.2)
- added R69: 10k, Resistor_SMD:R_0805_2012Metric, F.Cu at (438.4, 161.4)
- added R7: 10k, Resistor_SMD:R_0805_2012Metric, F.Cu at (234.0, 139.6)
- added R70: 1k, Resistor_SMD:R_0805_2012Metric, F.Cu at (420.9, 138.0)
- added R71: 10k, Resistor_SMD:R_0805_2012Metric, F.Cu at (424.4, 138.0)
- added R72: 10k, Resistor_SMD:R_0805_2012Metric, F.Cu at (430.7, 164.6)
- added R73: 600, Resistor_SMD:R_0805_2012Metric, F.Cu at (436.9, 139.6)
- added R74: 330, Resistor_SMD:R_0805_2012Metric, F.Cu at (441.0, 169.8)
- added R75: 10k, Resistor_SMD:R_0805_2012Metric, F.Cu at (426.3, 170.2)
- added R76: 330, Resistor_SMD:R_0805_2012Metric, F.Cu at (441.0, 172.0)
- added R77: 10k, Resistor_SMD:R_0805_2012Metric, F.Cu at (465.8, 139.6)
- added R78: 10k, Resistor_SMD:R_0805_2012Metric, F.Cu at (463.9, 161.2)
- added R79: 10k, Resistor_SMD:R_0805_2012Metric, F.Cu at (471.5, 161.4)
- added R8: 10k, Resistor_SMD:R_0805_2012Metric, F.Cu at (232.1, 161.2)
- added R80: 1k, Resistor_SMD:R_0805_2012Metric, F.Cu at (454.0, 138.0)
- added R81: 10k, Resistor_SMD:R_0805_2012Metric, F.Cu at (457.5, 138.0)
- added R82: 10k, Resistor_SMD:R_0805_2012Metric, F.Cu at (463.8, 164.6)
- added R83: 600, Resistor_SMD:R_0805_2012Metric, F.Cu at (470.0, 139.6)
- added R84: 330, Resistor_SMD:R_0805_2012Metric, F.Cu at (474.1, 169.8)
- added R85: 10k, Resistor_SMD:R_0805_2012Metric, F.Cu at (459.4, 170.2)
- added R86: 330, Resistor_SMD:R_0805_2012Metric, F.Cu at (474.1, 172.0)
- added R87: 10k, Resistor_SMD:R_0805_2012Metric, F.Cu at (504.8, 171.2)
- added R88: 10k, Resistor_SMD:R_0805_2012Metric, F.Cu at (504.8, 174.1)
- added R89: 10k, Resistor_SMD:R_0805_2012Metric, F.Cu at (504.8, 177.1)
- added R9: 10k, Resistor_SMD:R_0805_2012Metric, F.Cu at (239.7, 161.4)
- added R90: 10k, Resistor_SMD:R_0805_2012Metric, F.Cu at (504.8, 180.0)
- added R91: 10k, Resistor_SMD:R_0805_2012Metric, F.Cu at (504.8, 183.0)
- added R92: 330, Resistor_SMD:R_0805_2012Metric, F.Cu at (496.5, 171.2)
- added R93: 330, Resistor_SMD:R_0805_2012Metric, F.Cu at (496.5, 174.2)
- added R94: 330, Resistor_SMD:R_0805_2012Metric, F.Cu at (496.5, 177.2)
- added R95: 330, Resistor_SMD:R_0805_2012Metric, F.Cu at (496.5, 180.0)
- added R96: 330, Resistor_SMD:R_0805_2012Metric, F.Cu at (496.5, 183.0)
- added R97: 10k, Resistor_SMD:R_0805_2012Metric, F.Cu at (504.8, 185.9)
- added R98: 10k, Resistor_SMD:R_0805_2012Metric, F.Cu at (504.8, 188.9)
- added R99: 10k, Resistor_SMD:R_0805_2012Metric, F.Cu at (504.8, 191.8)
- added SW1: SW_SPDT, Button_Switch_SMD:SW_SPDT_CK_JS102011SAQN, F.Cu at (199.0, 206.2)
- added SW2: SW_Push, Button_Switch_SMD:SW_SPST_PTS647_Sx50, F.Cu at (171.4, 182.4)
- added T1: Transformer_1P_1S, Phones:TRAN6_SM-LP-5001_BRN, F.Cu at (236.0, 148.0)
- added T2: Transformer_1P_1S, Phones:TRAN6_SM-LP-5001_BRN, F.Cu at (269.1, 148.0)
- added T3: Transformer_1P_1S, Phones:TRAN6_SM-LP-5001_BRN, F.Cu at (302.2, 148.0)
- added T4: Transformer_1P_1S, Phones:TRAN6_SM-LP-5001_BRN, F.Cu at (335.3, 148.0)
- added T5: Transformer_1P_1S, Phones:TRAN6_SM-LP-5001_BRN, F.Cu at (368.5, 148.0)
- added T6: Transformer_1P_1S, Phones:TRAN6_SM-LP-5001_BRN, F.Cu at (401.6, 148.0)
- added T7: Transformer_1P_1S, Phones:TRAN6_SM-LP-5001_BRN, F.Cu at (434.7, 148.0)
- added T8: Transformer_1P_1S, Phones:TRAN6_SM-LP-5001_BRN, F.Cu at (467.8, 148.0)
- added TP1: TestPoint, Testpoints:M5_3in1_TestPoint, F.Cu at (241.8, 127.2)
- added TP10: TestPoint, Testpoints:M5_3in1_TestPoint, F.Cu at (274.9, 127.2)
- added TP11: TestPoint, Testpoints:M5_3in1_TestPoint, F.Cu at (261.3, 127.2)
- added TP12: TestPoint, Testpoints:M5_3in1_TestPoint, F.Cu at (270.3, 127.2)
- added TP13: TestPoint, Testpoints:M5_3in1_TestPoint, F.Cu at (265.8, 127.2)
- added TP14: TestPoint, Testpoints:M5_3in1_TestPoint, F.Cu at (273.8, 154.2)
- added TP15: TestPoint, Testpoints:M5_3in1_TestPoint, F.Cu at (260.3, 157.6)
- added TP16: TestPoint, Testpoints:M5_3in1_TestPoint, F.Cu at (276.7, 153.2)
- added TP17: TestPoint, Testpoints:M5_3in1_TestPoint, F.Cu at (259.5, 174.6)
- added TP18: TestPoint, Testpoints:M5_3in1_TestPoint, F.Cu at (264.5, 190.0)
- added TP19: TestPoint, Testpoints:M5_3in1_TestPoint, F.Cu at (308.0, 127.2)
- added TP2: TestPoint, Testpoints:M5_3in1_TestPoint, F.Cu at (228.2, 127.2)
- added TP20: TestPoint, Testpoints:M5_3in1_TestPoint, F.Cu at (294.4, 127.2)
- added TP21: TestPoint, Testpoints:M5_3in1_TestPoint, F.Cu at (303.5, 127.2)
- added TP22: TestPoint, Testpoints:M5_3in1_TestPoint, F.Cu at (298.9, 127.2)
- added TP23: TestPoint, Testpoints:M5_3in1_TestPoint, F.Cu at (306.9, 154.2)
- added TP24: TestPoint, Testpoints:M5_3in1_TestPoint, F.Cu at (293.4, 157.6)
- added TP25: TestPoint, Testpoints:M5_3in1_TestPoint, F.Cu at (309.8, 153.2)
- added TP26: TestPoint, Testpoints:M5_3in1_TestPoint, F.Cu at (292.6, 174.6)
- added TP27: TestPoint, Testpoints:M5_3in1_TestPoint, F.Cu at (297.6, 190.0)
- added TP28: TestPoint, Testpoints:M5_3in1_TestPoint, F.Cu at (341.1, 127.2)
- added TP29: TestPoint, Testpoints:M5_3in1_TestPoint, F.Cu at (327.5, 127.2)
- added TP3: TestPoint, Testpoints:M5_3in1_TestPoint, F.Cu at (237.2, 127.2)
- added TP30: TestPoint, Testpoints:M5_3in1_TestPoint, F.Cu at (336.6, 127.2)
- added TP31: TestPoint, Testpoints:M5_3in1_TestPoint, F.Cu at (332.0, 127.2)
- added TP32: TestPoint, Testpoints:M5_3in1_TestPoint, F.Cu at (340.0, 154.2)
- added TP33: TestPoint, Testpoints:M5_3in1_TestPoint, F.Cu at (326.5, 157.6)
- added TP34: TestPoint, Testpoints:M5_3in1_TestPoint, F.Cu at (342.9, 153.2)
- added TP35: TestPoint, Testpoints:M5_3in1_TestPoint, F.Cu at (325.7, 174.6)
- added TP36: TestPoint, Testpoints:M5_3in1_TestPoint, F.Cu at (330.8, 190.0)
- added TP37: TestPoint, Testpoints:M5_3in1_TestPoint, F.Cu at (374.2, 127.2)
- added TP38: TestPoint, Testpoints:M5_3in1_TestPoint, F.Cu at (360.6, 127.2)
- added TP39: TestPoint, Testpoints:M5_3in1_TestPoint, F.Cu at (369.7, 127.2)
- added TP4: TestPoint, Testpoints:M5_3in1_TestPoint, F.Cu at (232.7, 127.2)
- added TP40: TestPoint, Testpoints:M5_3in1_TestPoint, F.Cu at (365.1, 127.2)
- added TP41: TestPoint, Testpoints:M5_3in1_TestPoint, F.Cu at (373.1, 154.2)
- added TP42: TestPoint, Testpoints:M5_3in1_TestPoint, F.Cu at (359.6, 157.6)
- added TP43: TestPoint, Testpoints:M5_3in1_TestPoint, F.Cu at (376.0, 153.2)
- added TP44: TestPoint, Testpoints:M5_3in1_TestPoint, F.Cu at (358.8, 174.6)
- added TP45: TestPoint, Testpoints:M5_3in1_TestPoint, F.Cu at (363.9, 190.0)
- added TP46: TestPoint, Testpoints:M5_3in1_TestPoint, F.Cu at (407.3, 127.2)
- added TP47: TestPoint, Testpoints:M5_3in1_TestPoint, F.Cu at (393.7, 127.2)
- added TP48: TestPoint, Testpoints:M5_3in1_TestPoint, F.Cu at (402.8, 127.2)
- added TP49: TestPoint, Testpoints:M5_3in1_TestPoint, F.Cu at (398.3, 127.2)
- added TP5: TestPoint, Testpoints:M5_3in1_TestPoint, F.Cu at (240.6, 154.2)
- added TP50: TestPoint, Testpoints:M5_3in1_TestPoint, F.Cu at (406.2, 154.2)
- added TP51: TestPoint, Testpoints:M5_3in1_TestPoint, F.Cu at (392.7, 157.6)
- added TP52: TestPoint, Testpoints:M5_3in1_TestPoint, F.Cu at (409.1, 153.2)
- added TP53: TestPoint, Testpoints:M5_3in1_TestPoint, F.Cu at (391.9, 174.6)
- added TP54: TestPoint, Testpoints:M5_3in1_TestPoint, F.Cu at (397.0, 190.0)
- added TP55: TestPoint, Testpoints:M5_3in1_TestPoint, F.Cu at (440.4, 127.2)
- added TP56: TestPoint, Testpoints:M5_3in1_TestPoint, F.Cu at (426.8, 127.2)
- added TP57: TestPoint, Testpoints:M5_3in1_TestPoint, F.Cu at (435.9, 127.2)
- added TP58: TestPoint, Testpoints:M5_3in1_TestPoint, F.Cu at (431.4, 127.2)
- added TP59: TestPoint, Testpoints:M5_3in1_TestPoint, F.Cu at (439.3, 154.2)
- added TP6: TestPoint, Testpoints:M5_3in1_TestPoint, F.Cu at (227.2, 157.6)
- added TP60: TestPoint, Testpoints:M5_3in1_TestPoint, F.Cu at (425.8, 157.6)
- added TP61: TestPoint, Testpoints:M5_3in1_TestPoint, F.Cu at (442.2, 153.2)
- added TP62: TestPoint, Testpoints:M5_3in1_TestPoint, F.Cu at (425.0, 174.6)
- added TP63: TestPoint, Testpoints:M5_3in1_TestPoint, F.Cu at (430.1, 190.0)
- added TP64: TestPoint, Testpoints:M5_3in1_TestPoint, F.Cu at (473.6, 127.2)
- added TP65: TestPoint, Testpoints:M5_3in1_TestPoint, F.Cu at (460.0, 127.2)
- added TP66: TestPoint, Testpoints:M5_3in1_TestPoint, F.Cu at (469.0, 127.2)
- added TP67: TestPoint, Testpoints:M5_3in1_TestPoint, F.Cu at (464.5, 127.2)
- added TP68: TestPoint, Testpoints:M5_3in1_TestPoint, F.Cu at (472.4, 154.2)
- added TP69: TestPoint, Testpoints:M5_3in1_TestPoint, F.Cu at (459.0, 157.6)
- added TP7: TestPoint, Testpoints:M5_3in1_TestPoint, F.Cu at (243.6, 153.2)
- added TP70: TestPoint, Testpoints:M5_3in1_TestPoint, F.Cu at (475.4, 153.2)
- added TP71: TestPoint, Testpoints:M5_3in1_TestPoint, F.Cu at (458.2, 174.6)
- added TP72: TestPoint, Testpoints:M5_3in1_TestPoint, F.Cu at (463.2, 190.0)
- added TP73: TestPoint, Testpoints:M5_3in1_TestPoint, F.Cu at (481.6, 203.5)
- added TP74: TestPoint, Testpoints:M5_3in1_TestPoint, F.Cu at (481.6, 198.9)
- added TP75: TestPoint, Testpoints:M5_3in1_TestPoint, F.Cu at (481.6, 194.2)
- added TP76: TestPoint, Testpoints:M5_3in1_TestPoint, F.Cu at (481.6, 189.6)
- added TP77: TestPoint, Testpoints:M5_3in1_TestPoint, F.Cu at (481.6, 184.9)
- added TP78: TestPoint, Testpoints:M5_3in1_TestPoint, F.Cu at (481.6, 180.3)
- added TP79: TestPoint, Testpoints:M5_3in1_TestPoint, F.Cu at (481.6, 175.6)
- added TP8: TestPoint, Testpoints:M5_3in1_TestPoint, F.Cu at (226.4, 174.6)
- added TP80: TestPoint, Testpoints:M5_3in1_TestPoint, F.Cu at (481.6, 171.0)
- added TP81: TestPoint, Testpoints:M5_3in1_TestPoint, F.Cu at (481.6, 166.3)
- added TP82: TestPoint, Testpoints:M5_3in1_TestPoint, F.Cu at (481.6, 161.7)
- added TP83: TestPoint, Testpoints:M5_3in1_TestPoint, F.Cu at (481.6, 157.0)
- added TP84: TestPoint, Testpoints:M5_3in1_TestPoint, F.Cu at (481.6, 152.4)
- added TP85: TestPoint, Testpoints:M5_3in1_TestPoint, F.Cu at (172.8, 141.6)
- added TP86: TestPoint, Testpoints:M5_3in1_TestPoint, F.Cu at (177.5, 141.6)
- added TP87: TestPoint, Testpoints:M5_3in1_TestPoint, F.Cu at (182.1, 141.6)
- added TP88: TestPoint, Testpoints:M5_3in1_TestPoint, F.Cu at (186.8, 141.6)
- added TP89: TestPoint, Testpoints:M5_3in1_TestPoint, F.Cu at (191.4, 141.6)
- added TP9: TestPoint, Testpoints:M5_3in1_TestPoint, F.Cu at (231.4, 190.0)
- added TP90: TestPoint, Testpoints:M5_3in1_TestPoint, F.Cu at (196.1, 141.6)
- added TP91: TestPoint, Testpoints:M5_3in1_TestPoint, F.Cu at (200.7, 141.6)
- added TP92: TestPoint, Testpoints:M5_3in1_TestPoint, F.Cu at (205.4, 141.6)
- added TP93: TestPoint, Testpoints:M5_3in1_TestPoint, F.Cu at (172.8, 156.0)
- added TP94: TestPoint, Testpoints:M5_3in1_TestPoint, F.Cu at (177.5, 156.0)
- added TP95: TestPoint, Testpoints:M5_3in1_TestPoint, F.Cu at (182.1, 156.0)
- added U1: TPS2116DRL, Package_TO_SOT_SMD:SOT-583-8, F.Cu at (179.3, 192.4)
- added U2: AZ1117-3.3, Package_TO_SOT_SMD:SOT-223, F.Cu at (187.0, 189.9)
- added U3: STM32F303RETx, Package_QFP:LQFP-64_10x10mm_P0.5mm, F.Cu at (204.5, 174.2)
- added U4: TLV2372, Package_SO:SOIC-8_3.9x4.9mm_P1.27mm, F.Cu at (223.0, 131.9)
- added U5: TLV2372, Package_SO:SOIC-8_3.9x4.9mm_P1.27mm, F.Cu at (289.2, 131.9)
- added U6: TLV2372, Package_SO:SOIC-8_3.9x4.9mm_P1.27mm, F.Cu at (355.6, 132.0)
- added U7: TLV2372, Package_SO:SOIC-8_3.9x4.9mm_P1.27mm, F.Cu at (421.6, 131.8)
- added U8: 74LS165, Package_SO:TSSOP-16_4.4x5mm_P0.65mm, F.Cu at (487.0, 142.7)
- added U9: MCP3008, Package_SO:SOIC-16_3.9x9.9mm_P1.27mm, F.Cu at (203.6, 132.9)
- added Y1: 8M, Crystal:Crystal_SMD_Abracon_ABM3-2Pin_5.0x3.2mm_HandSoldering, F.Cu at (188.5, 175.9)
Routing:
- net GND: track 0.00 -> 108.3 mm, vias 0 -> 43
- net Net-(T3-AB): track 0.00 -> 94.3 mm, vias 0 -> 4
- net Net-(T1-AB): track 0.00 -> 94.3 mm, vias 0 -> 4
- net Net-(T8-AB): track 0.00 -> 94.3 mm, vias 0 -> 4
- net Net-(T7-AB): track 0.00 -> 94.3 mm, vias 0 -> 4
- net Net-(T6-AB): track 0.00 -> 94.3 mm, vias 0 -> 4
- net Net-(T5-AB): track 0.00 -> 94.3 mm, vias 0 -> 4
- net Net-(T4-AB): track 0.00 -> 94.3 mm, vias 0 -> 4
- net Net-(T2-AB): track 0.00 -> 94.3 mm, vias 0 -> 4
- net Net-(J13-Pad1): track 0.00 -> 83.3 mm
- net Net-(J11-Pad1): track 0.00 -> 83.3 mm
- net Net-(J7-Pad1): track 0.00 -> 83.3 mm
- net Net-(J5-Pad1): track 0.00 -> 83.3 mm
- net Net-(J10-Pad4): track 0.00 -> 83.3 mm
- net Net-(J19-Pad1): track 0.00 -> 83.3 mm
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- added copper zone on In1.Cu, net GND
Other:
- board outline added: 363.2 x 100.4 mm
- board text added: "+5V"
- board text added: "1"
- board text added: "2"
- board text added: "3"
- board text added: "4"
- board text added: "5"
- board text added: "6"
- board text added: "7"
- board text added: "74LS165 Shift Register"
- board text added: "8"
- board text added: "ADC Lines"
- board text added: "Boot Mode"
- board text added: "Button States"
- board text added: "Connectors"
- board text added: "Flash (Normal)"
- board text added: "GND"
- board text added: "Line 1"
- board text added: "Line 2"
- board text added: "Line 3"
- board text added: "Line 4"
- board text added: "Line 5"
- board text added: "Line 6"
- board text added: "Line 7"
- board text added: "Line 8"
- board text added: "M5 PBX Sniffer V2.1"
- board text added: "MCP3008 ADC"
- board text added: "Made with love by Tobe Cynar 2026/08/21"
- board text added: "Power Jack"
- board text added: "Reset Button"
- board text added: "SPI"
- board text added: "STM32F303RE"
- board text added: "SWD"
- board text added: "Signal Jack"
- board text added: "System Memory"
- board text added: "UART"
- board text added: "USB Power"
- board text added: "clk"
- board text added: "controlSW"
- board text added: "hookSW"
- board text added: "miso"
- board text added: "mosi"
