File: transferbtns.kicad_sch (KiCad schematic)
At the start: 23 parts, among them J1 8P8C, J2 8P8C, U6 74LS165

Commit message: unsplit grounds, finish power circuitry, start picking footprints/partnumbers
Parts:
- R1, R2, R3, R4, R5, R6, R7, R8: footprint Resistor_THT:R_Axial_DIN0207_L6.3mm_D2.5mm_P7.62mm_Horizontal -> Resistor_SMD:R_0805_2012Metric
Connections:
- net GNDD renamed GND
