File: linectrl.kicad_sch (KiCad schematic)
At the start: 1 part, among them U2 LM358

Commit message: added power mux, finished up schematic and picking footprints/partnumbers
Parts:
- removed U2: LM358, Package_DIP:DIP-8_W7.62mm, symbol Amplifier_Operational:LM358
- added C18: 100n, Capacitor_SMD:C_0805_2012Metric, symbol Device:C_Small
- added U4: TLV2372, Package_SO:SOIC-8_3.9x4.9mm_P1.27mm, symbol Amplifier_Operational:TLV2372
Connections:
- net +5VA: now also C18.1, U4.8 (V+)
- net GND: now also C18.2, U4.4 (V-)
- net LineCtrlSingle1/ampV+: now also U4.3 (+)
- net LineCtrlSingle1/ampV-: now also U4.2 (-)
- net LineCtrlSingle2/ampV+: now also U4.5 (+)
- net LineCtrlSingle2/ampV-: now also U4.6 (-)
- net audioOut1: now also U4.1
- net audioOut2: now also U4.7
